File: Karane_Kicad/Karane_Kicad.kicad_pcb (KiCad board)
At the start: 2 copper layers, 134 x 85 mm, 145 parts, among them J1 FFC, J11 Conn_01x02_Socket, J2 SerialWire, J3 FFC, J4 Conn_01x02_Socket, J5 Conn_01x02_Socket, J8 Conn_01x02_Socket, J9 Conn_01x02_Socket, Q1 AO3400A, SW1 SW_Push, SW2 SW_Push, SW3 SW_Push, SW4 SW_Push_SPDT, U1 QRE111GR, U10 QRE111GR, U11 QRE111GR, U12 QRE111GR, U13 QRE111GR, U14 QRE111GR, U15 QRE111GR, U16 QRE111GR, U17 QRE111GR, U18 MP6551GQB-P, U19 STM32f103C8t6, U2 CD74HC4067SM, U20 MP6551GQB-P, U21 AD8418, U22 AD8418, U23 MPU6500, U24 CN3903, U25 AS5145B, U26 AS5145B, U3 QRE111GR, U4 QRE111GR, U5 QRE111GR, U6 QRE111GR, U7 QRE111GR, U8 QRE111GR, U9 QRE111GR, Y1 8Mhz

Commit message: Agregado Mosfet dual
Parts:
- added C34: 1uF, Capacitor_SMD:C_0603_1608Metric_Pad1.08x0.95mm_HandSolder, F.Cu at (151.2, 94.3)
- added C35: 1uF, Capacitor_SMD:C_0603_1608Metric_Pad1.08x0.95mm_HandSolder, F.Cu at (151.2, 96.8)
- added J10: SQJ951EP, Package_SO:PowerPAK_SO-8_Dual, F.Cu at (153.5, 89.8)
- added R52: 100k, Resistor_SMD:R_0805_2012Metric_Pad1.20x1.40mm_HandSolder, F.Cu at (159.9, 88.0)
- added R53: 100k, Resistor_SMD:R_0805_2012Metric_Pad1.20x1.40mm_HandSolder, F.Cu at (159.9, 90.9)
- added U27: ME6211C33_regulador, Package_TO_SOT_SMD:SOT-23-5_HandSoldering, F.Cu at (156.3, 95.5)
- added Y2: Crystal_GND24, Crystal:Crystal_SMD_3225-4Pin_3.2x2.5mm, F.Cu at (182.8, 57.9)
- C30: value 10uF -> 100uF
- R42: value 100K -> 44K
- R43: value 39K -> 10K
- U21, U22: footprint Footprint:AD8418_soic -> Footprint:AD8418_MicroSoic
- moved G*** 165.3 mm to (249.0, 16.6)
- moved G*** 154.1 mm to (319.0, 7.30)
- moved G*** 143.8 mm to (290.2, 3.91)
Connections:
- net /encoder/ENCA_ML_CONN renamed /Encoder/ENCA_ML_CONN
- net /encoder/ENCA_MR_CONN renamed /Encoder/ENCA_MR_CONN
- net /encoder/ENCB_ML_CONN renamed /Encoder/ENCB_ML_CONN
- net /encoder/ENCB_MR_CONN renamed /Encoder/ENCB_MR_CONN
- net /encoder/ENCC_ML_CONN renamed /Encoder/ENCC_ML_CONN
- net /encoder/ENCC_MR_CONN renamed /Encoder/ENCC_MR_CONN
- net /encoder/GNDA_CONN renamed /Encoder/GNDA_CONN
- net /encoder/GNDB_CONN renamed /Encoder/GNDB_CONN
- net /encoder/VCCA_CONN renamed /Encoder/VCCA_CONN
- net /encoder/VCCB_CONN renamed /Encoder/VCCB_CONN
- C26 pad 1: +3.3V -> +5V
- C27 pad 1: +3.3V -> +5V
- C28 pad 1: +3.3V -> +5V
- C30 pad 1: +3.3V -> +5V
- C36 pad 1: Net-(J11-Pin_2) -> /VOLTAGE
- C37 pad 1: Net-(J11-Pin_2) -> /VOLTAGE
- J11 pad 2: Net-(J11-Pin_2) -> Net-(J10-D1)
- J9 pad 1: GND -> Net-(J10-D1)
- J9 pad 2: Net-(J11-Pin_2) -> /VOLTAGE
- L1 pad 2: +3.3V -> +5V
- R42 pad 2: +3.3V -> +5V
- SW4 pad 2: /VOLTAGE -> Net-(SW4-B)
- SW4 pad 3: Net-(J11-Pin_2) -> GND
Routing:
- net Net-(J11-Pin_2): vias 17 -> 0
- net GND: vias 71 -> 88

Commit message: Se actualizo las librerias
Parts:
- removed Y1: 8Mhz, Crystal:Crystal_SMD_3225-4Pin_3.2x2.5mm
- moved C32 124.9 mm to (233.3, 58.8)
- moved J13 124.9 mm to (233.8, 62.6)
- moved U26 124.9 mm to (233.8, 59.9)
- moved C33 124.9 mm to (235.1, 59.9)
- moved C34 78.5 mm to (72.7, 97.0)
- moved C35 78.5 mm to (72.7, 99.5)
- moved J10 78.5 mm to (75.0, 92.5)
- moved R52 78.5 mm to (81.5, 90.7)
- moved R53 78.5 mm to (81.5, 93.7)
- moved U27 78.5 mm to (77.8, 98.2)
- moved J2 75.3 mm to (252.5, 82.5)
- moved Y2 49.2 mm to (210.9, 98.3)
- moved C29 34.6 mm to (233.4, 68.0)
- moved C31 34.6 mm to (235.1, 69.1)
- moved J12 34.6 mm to (233.8, 71.9)
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Routing:
- net GND: track 397.2 -> 0.00 mm, vias 88 -> 0
- net +3.3V: track 349.5 -> 0.00 mm, vias 30 -> 0
- net /VOLTAGE_BATT: track 123.0 -> 0.00 mm, vias 2 -> 0
- net /PWMA_ML: track 120.3 -> 0.00 mm, vias 6 -> 0
- net /MOTOR_EN: track 117.0 -> 0.00 mm, vias 5 -> 0
- net /ENCC_ML: track 115.9 -> 0.00 mm, vias 1 -> 0
- net /ENCB_ML: track 115.2 -> 0.00 mm, vias 1 -> 0
- net /SENSOR_A_ML: track 111.6 -> 0.00 mm, vias 2 -> 0
- net /ENCA_ML: track 109.8 -> 0.00 mm, vias 1 -> 0
- net /PWMB_ML: track 87.8 -> 0.00 mm, vias 2 -> 0
- net /LED2: track 72.8 -> 0.00 mm, vias 2 -> 0
- net /LED4: track 67.9 -> 0.00 mm, vias 2 -> 0
- net /VOLTAGE: track 64.2 -> 0.00 mm, vias 16 -> 0
- net /S1_MUX: track 59.7 -> 0.00 mm, vias 2 -> 0
- net /OUT_MUX: track 57.1 -> 0.00 mm
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Other:
- board size 134 x 85 mm -> 150.9 x 85 mm
- copper layers 2 -> 4
