File: Karane_Kicad/Karane_Kicad.kicad_pcb (KiCad board)
At the start: 4 copper layers, 134 x 85 mm, 151 parts, among them J1 FFC, J10 SQJ951EP, J11 Conn_01x02_Socket, J2 SerialWire, J3 FFC, J4 Conn_01x02_Socket, J5 Conn_01x02_Socket, J8 Conn_01x02_Socket, J9 Conn_01x02_Socket, Q1 AO3400A, SW1 SW_Push, SW2 SW_Push, SW3 SW_Push, SW4 SW_Push_SPDT, U1 QRE111GR, U10 QRE111GR, U11 QRE111GR, U12 QRE111GR, U13 QRE111GR, U14 QRE111GR, U15 QRE111GR, U16 QRE111GR, U17 QRE111GR, U18 MP6551GQB-P, U19 STM32f103C8t6, U2 CD74HC4067SM, U20 MP6551GQB-P, U21 AD8418, U22 AD8418, U23 MPU6500, U24 CN3903, U25 AS5145B, U26 AS5145B, U27 ME6211C33_regulador, U3 QRE111GR, U4 QRE111GR, U5 QRE111GR, U6 QRE111GR, U7 QRE111GR, U8 QRE111GR, U9 QRE111GR, Y2 Crystal_GND24

Commit message: Agregado symbol de mosfet
Parts:
- removed J11, J9: Conn_01x02_Socket, Connector_Samtec_HPM_THT:Samtec_HPM-02-01-x-S_Straight_1x02_Pitch5.08mm
- added J14: XT30_BATT, Connector_AMASS:AMASS_XT30U-F_1x02_P5.0mm_Vertical, F.Cu at (6.05, 55.2)
- added J15: XT30_LIPO, Connector_AMASS:AMASS_XT30U-F_1x02_P5.0mm_Vertical, F.Cu at (11.5, 73.7)
- moved C15 63.9 mm to (68.0, 94.8)
- moved C16 63.9 mm to (71.5, 92.2)
- moved C19 63.9 mm to (53.0, 94.8)
- moved C25 63.9 mm to (60.0, 70.0)
- moved C30 63.9 mm to (62.2, 60.5)
- moved C32 63.9 mm to (50.5, 50.4)
- moved C36 63.9 mm to (41.0, 79.0)
- moved C37 63.9 mm to (39.2, 81.7)
- moved D2 63.9 mm to (74.0, 78.2)
- moved D4 63.9 mm to (77.0, 79.2)
- moved D6 63.9 mm to (68.2, 61.1)
- moved H3 63.9 mm to (31.6, 76.8)
- moved H4 63.9 mm to (31.6, 96.2)
- moved J13 63.9 mm to (51.0, 54.2)
- moved J5 63.9 mm to (66.8, 89.8)
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Other:
- outline, holes or cut-outs redrawn
- board text removed: "+"
- board text removed: "-"
- board text removed: "BAT"
- board text removed: "BOOT0"
- board text removed: "GND"
- board text removed: "ML"
- board text removed: "MOTOR"
- board text removed: "MR"
- board text removed: "RST"

Commit message: Cambio de f103 a f401
Parts:
- removed the J10 at (105.5, 94.8)
- removed the J15 at (11.5, 73.7)
- removed the R35 at (244.1, 91.0)
- removed the R52 at (112.0, 93.0)
- removed the R53 at (112.0, 96.0)
- removed the SW4 at (41.9, 59.4)
- removed the U18 at (64.5, 94.2)
- removed the U19 at (255.0, 98.2)
- removed the U20 at (243.8, 115.7)
- added C16: 4.7uF, Capacitor_SMD:C_0603_1608Metric_Pad1.08x0.95mm_HandSolder, F.Cu at (53.9, 165.8)
- added C17: 1uF, Capacitor_SMD:C_0603_1608Metric_Pad1.08x0.95mm_HandSolder, F.Cu at (53.9, 168.4)
- added C2: 10nF, Capacitor_SMD:C_0603_1608Metric_Pad1.08x0.95mm_HandSolder, F.Cu at (53.9, 170.9)
- added C5: 4.7uF, Capacitor_SMD:C_0603_1608Metric_Pad1.08x0.95mm_HandSolder, F.Cu at (53.9, 163.3)
- added D1: Inolux_IN-P55TATRGB, LED_SMD:LED_Inolux_IN-P55TATRGB_PLCC6_5.0x5.5mm_P1.8mm, F.Cu at (66.8, 160.2)
- added D7: LED, LED_SMD:LED_1206_3216Metric_Pad1.42x1.75mm_HandSolder, F.Cu at (65.6, 169.8)
- added D8: SS34, Diode_SMD:D_SMA, F.Cu at (66.7, 165.8)
- added D9: 12v, Diode_SMD:D_1206_3216Metric_Pad1.42x1.75mm_HandSolder, F.Cu at (119.8, 115.5)
- added J11: XT30_BATT, Connector_AMASS:AMASS_XT30U-F_1x02_P5.0mm_Vertical, F.Cu at (119.5, 121.8)
- added J12: SQJ951EP, Package_SO:PowerPAK_SO-8_Dual, F.Cu at (115.0, 115.5)
- added J13: SQJ951EP, Package_SO:PowerPAK_SO-8_Dual, F.Cu at (128.4, 115.5)
- added J2: ~, Footprint:usb_C_stm32, F.Cu at (180.0, 119.0)
- added J7: Motor_8520, Connector_PinHeader_2.54mm:PinHeader_1x02_P2.54mm_Vertical, F.Cu at (65.6, 149.3)
- added Q2: AO3400A, Package_TO_SOT_SMD:SOT-23, F.Cu at (70.4, 149.2)
- added R10: 220, Resistor_SMD:R_0805_2012Metric_Pad1.20x1.40mm_HandSolder, F.Cu at (49.4, 157.3)
- added R18: 220, Resistor_SMD:R_0805_2012Metric_Pad1.20x1.40mm_HandSolder, F.Cu at (49.4, 154.4)
- added R19: 10k, Resistor_SMD:R_0805_2012Metric_Pad1.20x1.40mm_HandSolder, F.Cu at (49.4, 166.2)
- added R3: 10K, Resistor_SMD:R_0805_2012Metric_Pad1.20x1.40mm_HandSolder, F.Cu at (49.4, 169.1)
- added R4: 10K, Resistor_SMD:R_0805_2012Metric_Pad1.20x1.40mm_HandSolder, F.Cu at (30.2, 123.2)
- added R5: 100, Resistor_SMD:R_0805_2012Metric_Pad1.20x1.40mm_HandSolder, F.Cu at (30.2, 127.4)
- added R55: 100k, Resistor_SMD:R_0805_2012Metric_Pad1.20x1.40mm_HandSolder, F.Cu at (122.9, 113.8)
- added R57: 100k, Resistor_SMD:R_0805_2012Metric_Pad1.20x1.40mm_HandSolder, F.Cu at (122.9, 117.2)
- added R8: 220, Resistor_SMD:R_0805_2012Metric_Pad1.20x1.40mm_HandSolder, F.Cu at (49.4, 163.2)
- added R9: 220, Resistor_SMD:R_0805_2012Metric_Pad1.20x1.40mm_HandSolder, F.Cu at (49.4, 160.3)
- added SW2: SW_Push, Button_Switch_SMD:SW_SPST_CK_RS282G05A3, F.Cu at (57.2, 159.5)
- added SW5: SW_Push_SPDT, Button_Switch_SMD:SW_SPDT_PCM12, F.Cu at (127.5, 122.8)
- added U1: vs1838, Connector_PinHeader_2.54mm:PinHeader_1x03_P2.54mm_Vertical, F.Cu at (33.2, 122.8)
- added U2: ~, Package_QFP:LQFP-64_10x10mm_P0.5mm, F.Cu at (342.1, 221.2)
- added U21: MP6551GQB-P, Footprint:MP6551, F.Cu at (76.9, 149.4)
- added U22: AD8418, Footprint:AD8418_MicroSoic, F.Cu at (78.6, 154.2)
- added U23: AD8418, Footprint:AD8418_MicroSoic, F.Cu at (78.6, 159.1)
- added U24: MP6551GQB-P, Footprint:MP6551, F.Cu at (81.1, 149.4)
- J14: value XT30_BATT -> XT30_LIPO
- moved J3 189.9 mm to (422.6, 75.1)
- moved J14 131.7 mm to (126.0, 109.6)
- moved C32 119.6 mm to (-10.5, 62.4)
- moved C33 119.6 mm to (-10.5, 64.9)
- moved U26 119.6 mm to (-5.45, 63.6)
- moved H4 107.3 mm to (137.7, 112.3)
- moved H3 106.1 mm to (137.7, 77.7)
- moved H1 105.5 mm to (172.3, 77.7)
- moved H2 103.1 mm to (172.3, 112.3)
- moved C6 20.6 mm to (158.4, 115.5)
- moved C10 20.6 mm to (152.0, 115.5)
- moved U3 20.6 mm to (155.0, 115.2)
- moved C8 20.6 mm to (156.8, 118.2)
- renumbered C8 to C1, C24 to C10, C13 to C11, C14 to C12, C12 to C13, C10 to C14, C11 to C15, C2 to C18, C1 to C19, C3 to C20, C4 to C21, C5 to C22, C19 to C23, C20 to C24, C15 to C25, C16 to C26, C17 to C27, C18 to C28, C36 to C29, C21 to C3, C37 to C30, C25 to C31, C34 to C32, C35 to C33, C26 to C34, C27 to C35, C28 to C36, C30 to C37, C29 to C38, C31 to C39, C9 to C4, C32 to C40, C33 to C41, C22 to C6, C6 to C7, C23 to C8, C7 to C9, D6 to D10, D1 to D2, D2 to D3, D3 to D4, D4 to D5, D5 to D6, J3 to J1, J4 to J10, J12 to J15, J13 to J16, J2 to J3, J6 to J4, J7 to J5, J8 to J6, J1 to J8, J5 to J9, R40 to R1, R46 to R11, R47 to R12, R48 to R13, R49 to R14, R44 to R15, R45 to R16, R50 to R17, R34 to R2, R8 to R20, R9 to R21, R1 to R22, R4 to R23, R6 to R24, R10 to R25, R11 to R26, R12 to R27, R2 to R28, R5 to R29, R7 to R30, R13 to R31, R20 to R32, R21 to R33, R14 to R34, R15 to R35, R16 to R36, R22 to R37, R23 to R38, R24 to R39, R17 to R40, R18 to R41, R19 to R42, R25 to R43, R26 to R44, R27 to R45, R28 to R46, R29 to R47, R3 to R48, R30 to R49, R31 to R50, R32 to R51, R33 to R52, R37 to R53, R38 to R54, R51 to R56, R39 to R58, R42 to R59, R41 to R6, R43 to R60, R36 to R7, SW2 to SW4, U11 to U10, U12 to U11, U8 to U12, U9 to U13, U10 to U14, U13 to U15, U2 to U16, U14 to U17, U15 to U18, U16 to U19, U17 to U20, U24 to U25, U27 to U26, U25 to U27, U26 to U28, U23 to U3, U5 to U4, U6 to U5, U1 to U6, U3 to U7, U4 to U8, U7 to U9, Y2 to Y1
Connections:
- net /BUTTON renamed /BUTTON_START
- D6 pad 2: /LED5 -> /LED_OK
- J14 pad 2: Net-(J10-D1) -> /VOLTAGE
Routing:
- net Net-(D9-K): track 0.00 -> 13.9 mm, vias 0 -> 6
- net Net-(SW5-A): track 0.00 -> 8.39 mm, vias 0 -> 2
- net GND: track 0.00 -> 1.75 mm, vias 0 -> 10
- net Net-(U3-REGOUT): track 0.00 -> 1.73 mm
- net Net-(J11-VCC): vias 0 -> 16
- net Net-(D9-A): vias 0 -> 29
- net /VOLTAGE: vias 0 -> 23
- net +3.3V: vias 0 -> 4
- added copper zone on F.Cu, net /VOLTAGE
- added copper zone on In2.Cu, net /VOLTAGE
- added copper zone on In1.Cu, net GND
- added copper zone on F.Cu, net Net-(D9-A)
- added copper zone on In2.Cu, net Net-(D9-A)
- added copper zone on F.Cu, net Net-(J11-VCC)
- added copper zone on In2.Cu, net Net-(J11-VCC)
Other:
- board size 134 x 85 mm -> 135 x 84.8 mm
- board text removed: "3V3 | RX | TX GND | SWDIO | SWCLK"

Commit message: planos de alimentacion hechos
Parts:
- removed the U21 at (58.0, 94.8)
- removed the U21 at (76.9, 149.4)
- removed the U22 at (78.6, 154.2)
- removed the U22 at (250.3, 115.2)
- added C42: 1uF, Capacitor_SMD:C_0603_1608Metric_Pad1.08x0.95mm_HandSolder, F.Cu at (215.4, 90.3)
- added C43: 1uF, Capacitor_SMD:C_0603_1608Metric_Pad1.08x0.95mm_HandSolder, F.Cu at (216.3, 92.8)
- added U21: MP6551GQB-P, Footprint:MP6551, F.Cu at (107.0, 100.5)
- added U22: AD8418, Footprint:AD8418_MicroSoic, F.Cu at (99.0, 101.5)
- added U29: ME6211C33_regulador, Package_TO_SOT_SMD:SOT-23-5_HandSoldering, F.Cu at (213.7, 93.5)
- J10, J9: footprint Connector_PinHeader_2.54mm:PinHeader_1x02_P2.54mm_Vertical -> Connector_Molex:Molex_SL_171971-0002_1x02_P2.54mm_Vertical
- moved C16 186.5 mm to (240.4, 164.6)
- moved U2 185.4 mm to (191.0, 113.8), turned to 180 degrees
- moved C5 182.2 mm to (235.7, 176.1)
- moved C17 174.3 mm to (228.0, 159.9), turned to 90 degrees
- moved C23 161.1 mm to (214.0, 101.5), turned to -90 degrees
- moved C24 159.9 mm to (96.0, 101.5), turned to 90 degrees
- moved C33 158.3 mm to (147.6, 73.8), turned to 90 degrees
- moved C32 153.0 mm to (142.1, 73.8), turned to -90 degrees
- moved U26 150.5 mm to (144.8, 73.0), turned to -90 degrees
- moved R19 147.8 mm to (181.8, 100.5), turned to -90 degrees
- moved U23 144.4 mm to (211.0, 101.5), turned to 90 degrees
- moved D8 135.8 mm to (182.5, 95.0), turned to -90 degrees
- moved U24 131.4 mm to (203.0, 100.5)
- moved J7 126.8 mm to (178.8, 92.0)
- moved Q2 124.5 mm to (185.0, 100.5)
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Connections:
- C10 pad 1: +3.3V -> +3.3VA
- C11 pad 1: +3.3V -> +3.3VA
- C12 pad 1: +3.3V -> +3.3VA
- C13 pad 1: +3.3V -> +3.3VA
- C14 pad 1: +3.3V -> +3.3VA
- C15 pad 1: +3.3V -> +3.3VA
- C16 pad 1: +3.3V -> +3.3VA
- C17 pad 1: +3.3V -> +3.3VA
- C23 pad 1: +3.3V -> +3.3VA
- C6 pad 1: +3.3V -> +3.3VA
- J10 pad 1: /Motores/MOTA_MR -> /Motores/MOTB_MR
- J10 pad 2: /Motores/MOTB_MR -> /Motores/MOTA_MR
- J2 pad 11: +3.3V -> +3.3VA
- J2 pad 2: +3.3V -> +3.3VA
- J3 pad 1: +3.3V -> +3.3VA
- J4 pad 2: +3.3V -> +3.3VA
- R54 pad 1: /Motores/MOTB_MR -> /Motores/SHUNT_SENSOR_MR
- R54 pad 2: /Motores/SHUNT_SENSOR_MR -> /Motores/MOTB_MR
- U2 pad 1: +3.3V -> +3.3VA
- U2 pad 13: +3.3V -> +3.3VA
- U2 pad 19: +3.3V -> +3.3VA
- U2 pad 32: +3.3V -> +3.3VA
- U2 pad 48: +3.3V -> +3.3VA
- U2 pad 64: +3.3V -> +3.3VA
- U23 pad 1: /Motores/MOTB_MR -> /Motores/SHUNT_SENSOR_MR
- U23 pad 6: +3.3V -> +3.3VA
- U23 pad 7: +3.3V -> +3.3VA
- U23 pad 8: /Motores/SHUNT_SENSOR_MR -> /Motores/MOTB_MR
- U24 pad 1: /Motores/SHUNT_SENSOR_MR -> /Motores/MOTA_MR
- U24 pad 10: /Motores/SHUNT_SENSOR_MR -> /Motores/MOTA_MR
- U24 pad 3: /Motores/MOTA_MR -> /Motores/SHUNT_SENSOR_MR
- U24 pad 8: /Motores/MOTA_MR -> /Motores/SHUNT_SENSOR_MR
- U3 pad 13: +3.3V -> +3.3VA
- U3 pad 8: +3.3V -> +3.3VA
Routing:
- net +3.3V: track 0.00 -> 82.4 mm, vias 4 -> 3
- net +5V: track 0.00 -> 31.8 mm, vias 0 -> 13
- net /ALIMENTACION/FN: track 0.00 -> 26.4 mm
- net +3.3VA: track 0.00 -> 11.9 mm, vias 0 -> 10
- net GND: track 1.75 -> 9.29 mm, vias 10 -> 45
- net Net-(U25-EN): track 0.00 -> 7.09 mm
- net Net-(Q1-D): track 0.00 -> 6.28 mm
- net Net-(U25-SW): track 0.00 -> 5.92 mm
- net /EN_SENSORES: track 0.00 -> 2.54 mm
- net Net-(U25-BST): track 0.00 -> 2.19 mm
- net /Motores/SHUNT_SENSOR_ML: track 0.00 -> 1.80 mm, vias 0 -> 17
- net /Motores/MOTA_ML: track 0.00 -> 1.50 mm, vias 0 -> 8
- net /VOLTAGE: vias 23 -> 56
- net /Motores/SHUNT_SENSOR_MR: vias 0 -> 17
- net /Motores/MOTB_MR: vias 0 -> 12
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- added copper zone on In2.Cu, net +3.3VA
- added copper zone on In2.Cu, net +5V
- added copper zone on F.Cu, net /Motores/MOTA_ML
- added copper zone on In2.Cu, net /Motores/MOTA_ML
- added copper zone on F.Cu, net /Motores/MOTA_MR
- added copper zone on In2.Cu, net /Motores/MOTA_MR
- added copper zone on F.Cu, net /Motores/MOTB_ML
- added copper zone on In2.Cu, net /Motores/MOTB_ML
- added copper zone on F.Cu, net /Motores/MOTB_MR
- added copper zone on In2.Cu, net /Motores/MOTB_MR
- added copper zone on F.Cu, net /Motores/SHUNT_SENSOR_ML
- added copper zone on In2.Cu, net /Motores/SHUNT_SENSOR_ML
- added copper zone on F.Cu, net /Motores/SHUNT_SENSOR_MR
- added copper zone on In2.Cu, net /Motores/SHUNT_SENSOR_MR
- added copper zone on F.Cu, net Net-(U25-SW)
Other:
- outline, holes or cut-outs redrawn

Commit message: mitada de componentes colocados
Parts:
- added C44: 100nF, Capacitor_SMD:C_0603_1608Metric_Pad1.08x0.95mm_HandSolder, F.Cu at (119.7, 104.0)
- SW1, SW2, SW3, SW4: footprint Button_Switch_SMD:SW_SPST_CK_RS282G05A3 -> Button_Switch_SMD:SW_Push_SPST_NO_Alps_SKRK
- moved R5 156.3 mm to (180.6, 84.9), turned to -52 degrees
- moved R4 153.2 mm to (177.5, 81.1), turned to 128 degrees
- moved R3 149.4 mm to (191.3, 122.6), turned to -90 degrees
- moved U1 147.3 mm to (175.0, 82.8), turned to 38 degrees
- moved C2 144.0 mm to (189.5, 122.4), turned to -90 degrees
- moved SW2 133.7 mm to (185.7, 122.5)
- moved R2 121.8 mm to (156.3, 123.1), turned to 90 degrees
- moved SW4 120.3 mm to (147.6, 123.1), turned to 0 degrees
- moved C4 119.0 mm to (151.5, 123.0)
- moved C1 118.6 mm to (158.4, 123.1)
- moved R7 118.0 mm to (153.7, 123.1)
- moved SW1 112.6 mm to (162.2, 123.1), turned to 0 degrees
- moved C30 107.2 mm to (138.3, 122.5), turned to -90 degrees
- moved C29 103.1 mm to (135.4, 120.5), turned to -90 degrees
- moved C5 91.0 mm to (180.5, 103.8), turned to 180 degrees
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Connections:
- C7 pad 1: /OSC_B -> /OSC_A
- C9 pad 1: /OSC_A -> /OSC_B
- U2 pad 14: /ENCA_ML -> /ENCA_MR
- U2 pad 15: /ENCB_ML -> /ENCB_MR
- U2 pad 16: /ENCC_ML -> /ENCC_MR
- U2 pad 21: /ENCA_MR -> /ENCA_ML
- U2 pad 22: unconnected-(U2-PA6-Pad22) -> /MOTOR_EN
- U2 pad 23: unconnected-(U2-PA7-Pad23) -> /EN_SENSORES
- U2 pad 26: /S2_MUX -> /S3_MUX
- U2 pad 27: /S3_MUX -> /S2_MUX
- U2 pad 28: /BUTTON_START -> unconnected-(U2-PB2/BOOT1-Pad28)
- U2 pad 29: /BUTTON_STOP -> unconnected-(U2-PB10-Pad29)
- U2 pad 54: /ENCC_MR -> /ENCC_ML
- U2 pad 55: /ENCB_MR -> /ENCB_ML
- U2 pad 56: /EN_SENSORES -> /BUTTON_STOP
- U2 pad 57: /MOTOR_EN -> /BUTTON_START
- U2 pad 58: /PWMB_MR -> /PWMB_ML
- U2 pad 59: /PWMA_MR -> /PWMA_ML
- U2 pad 61: /PWMB_ML -> /PWMB_MR
- U2 pad 62: /PWMA_ML -> /PWMA_MR
- U2 pad 8: /SENSOR_A_ML -> /SENSOR_A_MR
- U2 pad 9: /SENSOR_A_MR -> /SENSOR_A_ML
- Y1 pad 1: /OSC_B -> /OSC_A
- Y1 pad 3: /OSC_A -> /OSC_B
Routing:
- net /SENSOR_A_ML: track 0.00 -> 136.9 mm, vias 0 -> 2
- net /VOLTAGE_BATT: track 0.00 -> 113.8 mm, vias 0 -> 2
- net /OUT_MUX: track 0.00 -> 59.5 mm, vias 0 -> 2
- net /S3_MUX: track 0.00 -> 52.2 mm
- net /S1_MUX: track 0.00 -> 52.2 mm
- net /S2_MUX: track 0.00 -> 52.1 mm
- net /S0_MUX: track 0.00 -> 52.0 mm
- net /NRST: track 0.00 -> 45.1 mm, vias 0 -> 2
- net /BOOT0: track 0.00 -> 44.6 mm, vias 0 -> 2
- net /EN_SENSORES: track 2.54 -> 45.7 mm
- net /IR_36KHZ: track 0.00 -> 40.9 mm, vias 0 -> 1
- net /PWMA_MR: track 0.00 -> 39.3 mm, vias 0 -> 2
- net GND: track 9.29 -> 47.9 mm, vias 45 -> 60
- net /MOSI: track 0.00 -> 35.4 mm, vias 0 -> 2
- net /SCK: track 0.00 -> 35.0 mm, vias 0 -> 2
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
Commit message: finalizado pcb v2
Parts:
- removed C38, C40: 10nF, Capacitor_SMD:C_0603_1608Metric_Pad1.08x0.95mm_HandSolder
- removed J3: SerialWire, Connector_IDC:IDC-Header_2x03_P2.54mm_Vertical
- added JP1: Jumper_2_Open, Jumper:SolderJumper-2_P1.3mm_Open_RoundedPad1.0x1.5mm, B.Cu at (116.3, 81.5)
- added JP2: Jumper_2_Open, Jumper:SolderJumper-2_P1.3mm_Open_RoundedPad1.0x1.5mm, B.Cu at (188.8, 81.2)
- added R61: 10k, Resistor_SMD:R_0603_1608Metric_Pad0.98x0.95mm_HandSolder, B.Cu at (119.5, 82.2)
- added R62: 10k, Resistor_SMD:R_0603_1608Metric_Pad0.98x0.95mm_HandSolder, B.Cu at (191.8, 82.2)
- C39, C41: value 10nF -> 100nF; moved to B.Cu
- G***, SW1, SW4: moved to B.Cu
- J15, J16: footprint Footprint:as5145_mod_1.27 -> Footprint:AS5145_Mod; moved to B.Cu
- J4, J5: footprint Footprint:as5145_con_1.27 -> Footprint:AS5145_CONN_PCB
- U27, U28: value AS5145B -> MT6701CT; footprint Package_SO:SSOP-16_5.3x6.2mm_P0.65mm -> Package_SO:SO-8_3.9x4.9mm_P1.27mm; moved to F.Cu
- moved G*** 233.9 mm to (107.5, 107.1)
- moved R10 172.8 mm to (214.5, 106.5)
- moved R9 171.1 mm to (212.5, 108.5)
- moved R8 170.0 mm to (211.0, 110.5)
- moved G*** 167.0 mm to (110.4, 109.9)
- moved R18 163.2 mm to (209.0, 120.5), turned to 180 degrees
- moved D7 151.3 mm to (209.5, 123.0), turned to 180 degrees
- moved J16 143.6 mm to (191.2, 85.2), turned to 90 degrees
- moved U28 143.1 mm to (191.2, 80.2), turned to -90 degrees
- moved C41 142.3 mm to (191.8, 80.2), turned to 0 degrees
- moved D1 140.3 mm to (195.1, 103.3), turned to 180 degrees
- moved R11 139.3 mm to (97.5, 121.0), turned to 0 degrees
- moved C39 137.3 mm to (119.5, 80.5), turned to 0 degrees
- moved J15 136.8 mm to (118.8, 85.0), turned to 90 degrees
- moved U27 136.8 mm to (118.8, 80.0), turned to -90 degrees
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Connections:
- D1 pad 1: GND -> Net-(D1-KB)
- D1 pad 2: GND -> Net-(D1-KR)
- D1 pad 3: GND -> Net-(D1-KG)
- D1 pad 4: Net-(D1-AG) -> /PWM_BLUE
- D1 pad 5: Net-(D1-AR) -> /PWM_GREEN
- D1 pad 6: Net-(D1-AB) -> /PWM_RED
- J4 pad 2: +3.3VA -> +3.3V
- J5 pad 2: +3.3V -> +3.3VA
- R10 pad 1: Net-(D1-AB) -> Net-(D1-KG)
- R10 pad 2: /PWM_BLUE -> GND
- R2 pad 1: +3.3V -> +3.3VA
- R4 pad 1: +3.3V -> +3.3VA
- R5 pad 1: +3.3V -> +3.3VA
- R8 pad 1: Net-(D1-AG) -> Net-(D1-KB)
- R8 pad 2: /PWM_GREEN -> GND
- R9 pad 1: Net-(D1-AR) -> Net-(D1-KR)
- R9 pad 2: /PWM_RED -> GND
- SW2 pad 1: +3.3V -> +3.3VA
- SW3 pad 1: +3.3V -> +3.3VA
- SW4 pad 1: +3.3V -> +3.3VA
- U27 pad 1: unconnected-(U27-MagINCn-Pad1) -> /Encoder/VCCA_CONN
- U27 pad 2: unconnected-(U27-MagDECn-Pad2) -> Net-(JP1-B)
- U27 pad 3: /Encoder/ENCA_ML_CONN -> unconnected-(U27-OUT-Pad3)
- U27 pad 4: /Encoder/ENCB_ML_CONN -> /Encoder/GNDA_CONN
- U27 pad 6: /Encoder/ENCC_ML_CONN -> /Encoder/ENCA_ML_CONN
- U27 pad 7: /Encoder/GNDA_CONN -> /Encoder/ENCB_ML_CONN
- U27 pad 8: unconnected-(U27-PDIO-Pad8) -> /Encoder/ENCC_ML_CONN
- U28 pad 1: unconnected-(U28-MagINCn-Pad1) -> /Encoder/VCCB_CONN
- U28 pad 2: unconnected-(U28-MagDECn-Pad2) -> Net-(JP2-B)
- U28 pad 3: /Encoder/ENCA_MR_CONN -> unconnected-(U28-OUT-Pad3)
- U28 pad 4: /Encoder/ENCB_MR_CONN -> /Encoder/GNDB_CONN
- U28 pad 6: /Encoder/ENCC_MR_CONN -> /Encoder/ENCA_MR_CONN
- U28 pad 7: /Encoder/GNDB_CONN -> /Encoder/ENCB_MR_CONN
- U28 pad 8: unconnected-(U28-PDIO-Pad8) -> /Encoder/ENCC_MR_CONN
Routing:
- net /MOTOR_EN: track 23.2 -> 157.8 mm, vias 0 -> 7
- net /LED1: track 0.00 -> 99.9 mm, vias 0 -> 4
- net /ENCC_ML: track 0.00 -> 98.6 mm, vias 0 -> 2
- net /ENCB_ML: track 0.00 -> 98.5 mm, vias 0 -> 2
- net /ENCA_ML: track 0.00 -> 93.7 mm, vias 0 -> 3
- net /PWMA_ML: track 0.00 -> 92.4 mm, vias 0 -> 2
- net /LED2: track 0.00 -> 92.2 mm, vias 0 -> 4
- net /PWMB_ML: track 0.00 -> 92.0 mm, vias 0 -> 2
- net /LED3: track 0.00 -> 59.9 mm
- net +3.3VA: track 28.7 -> 77.8 mm, vias 15 -> 19
- net /LED_ALARMA: track 0.00 -> 38.4 mm, vias 0 -> 6
- net /LED_OK: track 0.00 -> 35.0 mm, vias 0 -> 4
- net /SENSOR_A_MR: track 0.00 -> 29.2 mm, vias 0 -> 4
- net /PWM_BLUE: track 0.00 -> 28.8 mm, vias 0 -> 4
- net GND: track 47.9 -> 75.5 mm, vias 60 -> 70
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Other:
- board size 135 x 84.8 mm -> 135 x 78.5 mm
