File: Karane_Kicad/Karane_Kicad.kicad_pcb (KiCad board)
At the start: 4 copper layers, 135 x 78.5 mm, 177 parts, among them J1 FFC, J10 Conn_01x02_Socket, J11 XT30_BATT, J12 SQJ951EP, J13 SQJ951EP, J14 XT30_LIPO, J6 Conn_01x02_Socket, J7 Motor_8520, J8 FFC, J9 Conn_01x02_Socket, Q1 AO3400A, Q2 AO3400A, SW1 SW_Push, SW2 SW_Push, SW3 SW_Push, SW4 SW_Push, SW5 SW_Push_SPDT, U1 vs1838, U10 QRE111GR, U11 QRE111GR, U12 QRE111GR, U13 QRE111GR, U14 QRE111GR, U15 QRE111GR, U16 CD74HC4067SM, U17 QRE111GR, U18 QRE111GR, U19 QRE111GR, U20 QRE111GR, U21 MP6551GQB-P, U22 AD8418, U23 AD8418, U24 MP6551GQB-P, U25 CN3903, U26 ME6211C33_regulador, U27 MT6701CT, U28 MT6701CT, U29 ME6211C33_regulador, U3 MPU6500, U4 QRE111GR, U5 QRE111GR, U6 QRE111GR, U7 QRE111GR, U8 QRE111GR, U9 QRE111GR, Y1 Crystal_GND24

Commit message: agregado etiquetas
Parts:
- added kibuzzard-69E2B1AE: G***, kibuzzard-69E2B1AE, F.Cu at (100.8, 112.0)
- added kibuzzard-69E2B1AE: G***, kibuzzard-69E2B1AE, F.Cu at (189.0, 102.2)
- added kibuzzard-69E2B1FC: G***, kibuzzard-69E2B1FC, F.Cu at (100.5, 113.5)
- added kibuzzard-69E2B208: G***, kibuzzard-69E2B208, F.Cu at (100.8, 115.0)
- added kibuzzard-69E2B20B: G***, kibuzzard-69E2B20B, F.Cu at (100.8, 116.5)
- added kibuzzard-69E2B212: G***, kibuzzard-69E2B212, F.Cu at (100.8, 118.0)
- added kibuzzard-69E2B220: G***, kibuzzard-69E2B220, F.Cu at (208.8, 118.0)
- added kibuzzard-69E2B227: G***, kibuzzard-69E2B227, F.Cu at (209.0, 116.5)
- added kibuzzard-69E2B22F: G***, kibuzzard-69E2B22F, F.Cu at (208.9, 115.0)
- added kibuzzard-69E2B236: G***, kibuzzard-69E2B236, F.Cu at (208.9, 113.5)
- added kibuzzard-69E2B23E: G***, kibuzzard-69E2B23E, F.Cu at (208.9, 112.0)
- added kibuzzard-69E2B2B1: G***, kibuzzard-69E2B2B1, F.Cu at (196.0, 99.2)
- added kibuzzard-69E2B2B1: G***, kibuzzard-69E2B2B1, F.Cu at (135.5, 115.8)
- added kibuzzard-69E2B2B1: G***, kibuzzard-69E2B2B1, F.Cu at (114.0, 99.5)
- added kibuzzard-69E2B2B1: G***, kibuzzard-69E2B2B1, F.Cu at (135.5, 88.0)
- added kibuzzard-69E2B33D: G***, kibuzzard-69E2B33D, F.Cu at (180.2, 97.5)
- added kibuzzard-69E2B382: G***, kibuzzard-69E2B382, F.Cu at (186.8, 102.2)
- added kibuzzard-69E2B3C8: G***, kibuzzard-69E2B3C8, B.Cu at (211.5, 122.8)
- added kibuzzard-69E2B437: G***, kibuzzard-69E2B437, B.Cu at (167.8, 123.2)
- added kibuzzard-69E2B43D: G***, kibuzzard-69E2B43D, B.Cu at (143.0, 123.0)

Commit message: Agregado agujeros a pcb
Parts:
- added H5: MountingHole_Pad, MountingHole:MountingHole_2.2mm_M2_ISO14580_Pad, F.Cu at (220.0, 98.0)
- added H6: MountingHole_Pad, MountingHole:MountingHole_2.2mm_M2_ISO14580_Pad, F.Cu at (220.0, 121.0)
- added H7: MountingHole_Pad, MountingHole:MountingHole_2.2mm_M2_ISO14580_Pad, F.Cu at (90.0, 98.0)
- added H8: MountingHole_Pad, MountingHole:MountingHole_2.2mm_M2_ISO14580_Pad, F.Cu at (90.0, 121.0)
