File: Karane_Kicad/Sensores.kicad_sch (KiCad schematic)
At the start: 56 parts, among them J1 FFC, U1 QRE111GR, U10 QRE111GR, U11 QRE111GR, U12 QRE111GR, U13 QRE111GR, U14 QRE111GR, U15 QRE111GR, U16 QRE111GR, U17 QRE111GR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

Commit message: Cambio de f103 a f401
Parts:
- renumbered C2 to C18, C1 to C19, C3 to C20, C4 to C21, C5 to C22, J1 to J8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
