File: Karane_Kicad/Motores.kicad_sch (KiCad schematic)
At the start: 14 parts, among them J4 Conn_01x02_Socket, J5 Conn_01x02_Socket, U18 MP6551GQB-P, U20 MP6551GQB-P, U21 AD8418, U22 AD8418

Commit message: Agregado Mosfet dual
Parts:
- U21, U22: footprint Footprint:AD8418_soic -> Footprint:AD8418_MicroSoic

Commit message: Cambio de f103 a f401
Parts:
- removed U18, U20: MP6551GQB-P, Footprint:MP6551, symbol Micromouse_Library:MP6551GQB-P
- removed U21, U22: AD8418, Footprint:AD8418_MicroSoic, symbol Micromouse_Library:AD8418
- added U21, U24: MP6551GQB-P, Footprint:MP6551, symbol MOTORES_DRIVERS:MP6551GQB-P
- added U22, U23: AD8418, Footprint:AD8418_MicroSoic, symbol MOTORES_DRIVERS:AD8418
- renumbered C19 to C23, C20 to C24, C15 to C25, C16 to C26, C17 to C27, C18 to C28, J4 to J10, J5 to J9, R37 to R53, R38 to R54
Connections:
- net +3.3V: now also U22.6 (VDD), U22.7 (VREF1), U23.6 (VDD), U23.7 (VREF1)
- net BATT: now also U21.2 (VBATT), U24.2 (VBATT)
- net EN_MOTOR: now also U21.14 (EN1), U21.4 (EN2), U24.14 (EN1), U24.4 (EN2)
- net GND: now also U21.6 (SR), U21.9 (GND), U22.2 (GND), U22.3 (VREF2), U23.2 (GND), U23.3 (VREF2), U24.6 (SR), U24.9 (GND)
- net MOTA_ML: now also U21.3 (OUT2), U21.8 (OUT2)
- net MOTA_MR: now also U24.3 (OUT2), U24.8 (OUT2)
- net MOTB_ML: now also U22.1 (-IN)
- net MOTB_MR: now also U23.1 (-IN)
- net PWMA_ML: now also U21.13 (IN_1)
- net PWMA_MR: now also U24.13 (IN_1)
- net PWMB_ML: now also U21.5 (IN2)
- net PWMB_MR: now also U24.5 (IN2)
- net SENSOR_A_ML: now also U22.5 (OUT)
- net SENSOR_A_MR: now also U23.5 (OUT)
- net SHUNT_SENSOR_ML: now also U21.1 (OUT1), U21.10 (OUT1), U22.8 (+IN)
- net SHUNT_SENSOR_MR: now also U23.8 (+IN), U24.1 (OUT1), U24.10 (OUT1)

Commit message: planos de alimentacion hechos
Parts:
- J10, J9: footprint Connector_PinHeader_2.54mm:PinHeader_1x02_P2.54mm_Vertical -> Connector_Molex:Molex_SL_171971-0002_1x02_P2.54mm_Vertical
Connections:
- net +3.3V: no longer C23.1, U23.6 (VDD), U23.7 (VREF1)
- net MOTA_MR: now also J10.2 (Pin_2), U24.1 (OUT1), U24.10 (OUT1); no longer J10.1 (Pin_1), U24.3 (OUT2), U24.8 (OUT2)
- net MOTB_MR: now also J10.1 (Pin_1), R54.2, U23.8 (+IN); no longer J10.2 (Pin_2), R54.1, U23.1 (-IN)
- net SHUNT_SENSOR_MR: now also R54.1, U23.1 (-IN), U24.3 (OUT2), U24.8 (OUT2); no longer R54.2, U23.8 (+IN), U24.1 (OUT1), U24.10 (OUT1)
- new net +3.3VA: C23.1, U23.6 (VDD), U23.7 (VREF1)
Changed lines of the file:
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@@
-	)
-	(junction
-		(at 50.8 118.11)
-		(diameter 0)
-		(color 0 0 0 0)
 	)
 	(junction
@@
 	(wire
 		(pts
-			(xy 219.71 34.29) (xy 219.71 54.61)
-		)
-		(stroke
-			(width 0)
-			(type default)
-		)
-	)
-	(wire
-		(pts
-			(xy 44.45 118.11) (xy 50.8 118.11)
+			(xy 219.71 43.18) (xy 219.71 54.61)
 		)
 		(stroke
@@
 	(wire
 		(pts
-			(xy 227.33 44.45) (xy 227.33 54.61)
-		)
-		(stroke
-			(width 0)
-			(type default)
-		)
-	)
-	(wire
-		(pts
 			(xy 67.31 162.56) (xy 71.12 162.56)
 		)
@@
 	(wire
 		(pts
-			(xy 227.33 80.01) (xy 227.33 90.17)
-		)
-		(stroke
-			(width 0)
-			(type default)
-		)
-	)
-	(wire
-		(pts
 			(xy 165.1 26.67) (xy 177.8 26.67)
 		)
@@
 	(wire
 		(pts
-			(xy 219.71 80.01) (xy 219.71 99.06)
+			(xy 219.71 80.01) (xy 219.71 91.44)
 		)
 		(stroke
@@
 	(wire
 		(pts
-			(xy 57.15 118.11) (xy 50.8 118.11)
-		)
-		(stroke
-			(width 0)
-			(type default)
-		)
-	)
-	(wire
-		(pts
 			(xy 220.98 144.78) (xy 220.98 140.97)
 		)
@@
 	(wire
 		(pts
+			(xy 227.33 80.01) (xy 227.33 99.06)
+		)
+		(stroke
+			(width 0)
+			(type default)
+		)
+	)
+	(wire
+		(pts
 			(xy 73.66 81.28) (xy 73.66 100.33)
 		)
@@
 	(wire
 		(pts
-			(xy 50.8 118.11) (xy 50.8 115.57)
-		)
-		(stroke
-			(width 0)
-			(type default)
-		)
-	)
-	(wire
-		(pts
 			(xy 58.42 69.85) (xy 62.23 69.85)
 		)
@@
 	(wire
 		(pts
+			(xy 227.33 34.29) (xy 227.33 54.61)
+		)
+		(stroke
+			(width 0)
+			(type default)
+		)
+	)
+	(wire
+		(pts
 			(xy 77.47 50.8) (xy 77.47 55.88)
 		)
@@
 	(wire
 		(pts
-			(xy 44.45 119.38) (xy 44.45 118.11)
-		)
-		(stroke
-			(width 0)
-			(type default)
-		)
-	)
-	(wire
-		(pts
 			(xy 195.58 140.97) (xy 198.12 140.97)
 		)
@@
 		(pts
 			(xy 194.31 124.46) (xy 194.31 137.16)
+		)
+		(stroke
+			(width 0)
+			(type default)
+		)
+	)
+	(wire
+		(pts
+			(xy 44.45 116.84) (xy 44.45 119.38)
 		)
 		(stroke
@@
 	)
 	(label "SHUNT_SENSOR_MR"
-		(at 233.68 137.16 0)
+		(at 175.26 137.16 0)
 		(effects
 			(font
@@
 	)
 	(label "SHUNT_SENSOR_MR"
-		(at 219.71 34.29 270)
+		(at 227.33 34.29 270)
 		(effects
 			(font
@@
 	)
 	(label "MOTA_MR"
-		(at 227.33 90.17 90)
+		(at 219.71 91.44 90)
 		(effects
 			(font
@@
 	)
 	(label "SHUNT_SENSOR_MR"
-		(at 219.71 99.06 90)
+		(at 227.33 99.06 90)
 		(effects
 			(font
@@
 	)
 	(label "MOTB_MR"
-		(at 236.22 111.76 0)
+		(at 236.22 109.22 0)
 		(effects
 			(font
@@
 	)
 	(label "MOTA_MR"
-		(at 227.33 44.45 270)
+		(at 219.71 43.18 270)
 		(effects
 			(font
@@
 	)
 	(label "MOTB_MR"
-		(at 175.26 137.16 180)
+		(at 233.68 137.16 180)
 		(effects
 			(font
@@
 	)
 	(label "MOTA_MR"
-		(at 236.22 109.22 0)
+		(at 236.22 111.76 0)
 		(effects
 			(font
@@
 			)
 		)
-		(property "Footprint" "Connector_PinHeader_2.54mm:PinHeader_1x02_P2.54mm_Vertical"
+		(property "Footprint" "Connector_Molex:Molex_SL_171971-0002_1x02_P2.54mm_Vertical"
 			(at 113.03 118.11 0)
 			(hide yes)
@@
 			)
 		)
-		(property "Footprint" "Connector_PinHeader_2.54mm:PinHeader_1x02_P2.54mm_Vertical"
+		(property "Footprint" "Connector_Molex:Molex_SL_171971-0002_1x02_P2.54mm_Vertical"
 			(at 250.19 109.22 0)
 			(hide yes)
@@
 	(symbol
 		(lib_id "power:+3.3V")
-		(at 50.8 115.57 0)
+		(at 57.15 118.11 0)
 		(unit 1)
 		(body_style 1)
@@
 		(fields_autoplaced yes)
 		(property "Reference" "#PWR054"
-			(at 50.8 119.38 0)
+			(at 57.15 121.92 0)
 			(hide yes)
 			(show_name no)
@@
 		)
 		(property "Value" "+3.3V"
-			(at 50.8 110.49 0)
+			(at 57.15 113.03 0)
 			(show_name no)
 			(do_not_autoplace no)
@@
 		)
 		(property "Footprint" ""
-			(at 50.8 115.57 0)
+			(at 57.15 118.11 0)
 			(hide yes)
 			(show_name no)
@@
 		)
 		(property "Datasheet" ""
-			(at 50.8 115.57 0)
+			(at 57.15 118.11 0)
 			(hide yes)
 			(show_name no)
@@
 		)
 		(property "Description" "Power symbol creates a global label with name \"+3.3V\""
-			(at 50.8 115.57 0)
+			(at 57.15 118.11 0)
 			(hide yes)
 			(show_name no)
@@
 	)
 	(symbol
+		(lib_id "power:+3.3VA")
+		(at 44.45 116.84 0)
+		(unit 1)
+		(body_style 1)
+		(exclude_from_sim no)
+		(in_bom yes)
+		(on_board yes)
+		(in_pos_files yes)
+		(dnp no)
+		(fields_autoplaced yes)
+		(property "Reference" "#PWR091"
+			(at 44.45 120.65 0)
+			(hide yes)
+			(show_name no)
+			(do_not_autoplace no)
+			(effects
+				(font
+					(size 1.27 1.27)
+				)
+			)
+		)
+		(property "Value" "+3.3VA"
+			(at 44.45 111.76 0)
+			(show_name no)
+			(do_not_autoplace no)
+			(effects
+				(font
+					(size 1.27 1.27)
+				)
+			)
+		)
+		(property "Footprint" ""
+			(at 44.45 116.84 0)
+			(hide yes)
+			(show_name no)
+			(do_not_autoplace no)
+			(effects
+				(font
+					(size 1.27 1.27)
+				)
+			)
+		)
+		(property "Datasheet" ""
+			(at 44.45 116.84 0)
+			(hide yes)
+			(show_name no)
+			(do_not_autoplace no)
+			(effects
+				(font
+					(size 1.27 1.27)
+				)
+			)
+		)
+		(property "Description" "Power symbol creates a global label with name \"+3.3VA\""
+			(at 44.45 116.84 0)
+			(hide yes)
+			(show_name no)
+			(do_not_autoplace no)
+			(effects
+				(font
+					(size 1.27 1.27)
+				)
+			)
+		)
+		(pin "1"
+		)
+		(instances
+			(project "Karane_Kicad"
+				(path "/65dfbecc-0fbf-480c-951c-b0d4a210bc14/7b893f59-ff4a-45a4-9e11-7ed86a86e4e9"
+					(reference "#PWR091")
+					(unit 1)
+				)
+			)
+		)
+	)
+	(symbol
 		(lib_id "Device:R")
 		(at 81.28 149.86 90)
@@
 	)
 	(symbol
-		(lib_id "power:+3.3V")
+		(lib_id "power:+3.3VA")
 		(at 223.52 140.97 270)
 		(unit 1)
@@
 		(dnp no)
 		(fields_autoplaced yes)
-		(property "Reference" "#PWR063"
+		(property "Reference" "#PWR090"
 			(at 219.71 140.97 0)
 			(hide yes)
@@
 			)
 		)
-		(property "Value" "+3.3V"
+		(property "Value" "+3.3VA"
 			(at 227.33 140.9699 90)
 			(show_name no)
@@
 			)
 		)
-		(property "Description" "Power symbol creates a global label with name \"+3.3V\""
+		(property "Description" "Power symbol creates a global label with name \"+3.3VA\""
 			(at 223.52 140.97 0)
 			(hide yes)
@@
 			(project "Karane_Kicad"
 				(path "/65dfbecc-0fbf-480c-951c-b0d4a210bc14/7b893f59-ff4a-45a4-9e11-7ed86a86e4e9"
-					(reference "#PWR063")
+					(reference "#PWR090")
 					(unit 1)
 				)
