File: Inda_Kicad/ALIMENTACION.kicad_sch (KiCad schematic)
At the start: 28 parts, among them J11 XT30_BATT, J12 SQJ951EP, J13 SQJ951EP, J14 XT30_LIPO, SW5 SW_Push_SPDT, U25 CN3903, U26 ME6211C33_regulador, U29 ME6211C33_regulador

Commit message: kicad cambios
Parts:
- removed D9: 12v, Diode_SMD:D_1206_3216Metric_Pad1.42x1.75mm_HandSolder, symbol Device:D_Zener
- removed J12: SQJ951EP, Package_SO:PowerPAK_SO-8_Dual, symbol Micromouse_Library:SQJ951EP-T1_BE3
- removed J14: XT30_LIPO, Connector_AMASS:AMASS_XT30U-F_1x02_P5.0mm_Vertical, symbol Micromouse_Library:Conector_XT30
- removed R55: 100k, Resistor_SMD:R_0805_2012Metric_Pad1.20x1.40mm_HandSolder, symbol Device:R
Connections:
- net at J11.2 (VCC): now also J13.1 (S1), J13.3 (S2), R57.1
- net at R57.2, SW5.1 (A): now also J13.2 (G1), J13.4 (G2)
Other:
- moved on the sheet: J11, R57
