File: Inda_Kicad/ALIMENTACION.kicad_sch (KiCad schematic)
At the start: 24 parts, among them J11 XT30_BATT, J13 SQJ951EP, SW5 SW_Push_SPDT, U25 CN3903, U26 ME6211C33_regulador, U29 ME6211C33_regulador

Commit message: Seguidor V3 con turbina finalizado a espera de revision
Parts:
- removed C29: 10uF, Capacitor_Tantalum_SMD:CP_EIA-6032-15_Kemet-U_HandSolder, symbol Device:C_Polarized
- removed C30, C31, C34, C35: 100nF, Capacitor_SMD:C_0603_1608Metric_Pad1.08x0.95mm_HandSolder, symbol Device:C
- removed C36: 22uF, Capacitor_SMD:C_0603_1608Metric_Pad1.08x0.95mm_HandSolder, symbol Device:C
- removed C37: 100uF, Capacitor_Tantalum_SMD:CP_EIA-6032-15_Kemet-U_HandSolder, symbol Device:C_Polarized
- removed D10: LED, LED_SMD:LED_1206_3216Metric_Pad1.42x1.75mm_HandSolder, symbol Device:LED
- removed J11: XT30_BATT, Connector_AMASS:AMASS_XT30U-F_1x02_P5.0mm_Vertical, symbol Micromouse_Library:Conector_XT30
- removed J13: SQJ951EP, Package_SO:PowerPAK_SO-8_Dual, symbol Micromouse_Library:SQJ951EP-T1_BE3
- removed R56: 220, Resistor_SMD:R_0805_2012Metric_Pad1.20x1.40mm_HandSolder, symbol Device:R
- removed R58, R60: 10K, Resistor_SMD:R_0805_2012Metric_Pad1.20x1.40mm_HandSolder, symbol Device:R
- removed R59: 44K, Resistor_SMD:R_0805_2012Metric_Pad1.20x1.40mm_HandSolder, symbol Device:R
- removed SW5: SW_Push_SPDT, Button_Switch_SMD:SW_SPDT_PCM12, symbol Switch:SW_Push_SPDT
- removed U25: CN3903, Package_SO:HSOP-8-1EP_3.9x4.9mm_P1.27mm_EP2.41x3.1mm, symbol Micromouse_Library:CN3903
- removed U26, U29: ME6211C33_regulador, Package_TO_SOT_SMD:SOT-23-5_HandSoldering, symbol Micromouse_Library:ME6211C33_regulador
- added C45: 0.1uF, Capacitor_SMD:C_0603_1608Metric, symbol Device:C
- added C46, C47: 22uF, Capacitor_Tantalum_SMD:CP_EIA-3528-15_AVX-H_HandSolder, symbol Device:C_Polarized
- added C48: 22uF, Capacitor_SMD:C_0603_1608Metric, symbol Device:C
- added C49, C51: 10uF, Capacitor_Tantalum_SMD:CP_EIA-3528-15_AVX-H_HandSolder, symbol Device:C_Polarized
- added C50, C52: 100nF, Capacitor_SMD:C_0603_1608Metric, symbol Device:C
- added D13: 12V, Resistor_SMD:R_1206_3216Metric_Pad1.30x1.75mm_HandSolder, symbol Device:D_Zener
- added D14: GREEN, LED_SMD:LED_1206_3216Metric_Pad1.42x1.75mm_HandSolder, symbol Device:LED
- added J14: XT30, Footprint:XT30U-F_1x02_P5.0mm_Vertical, symbol LIB_CONECTORES:Conector_XT30
- added J6: SQJ951EP, Package_SO:PowerPAK_SO-8_Dual, symbol LIB_MOSFET_BJT:SQJ951EP-T1_BE3
- added R63: 200K, Resistor_SMD:R_0603_1608Metric_Pad0.98x0.95mm_HandSolder, symbol Device:R
- added R64: 100k, Resistor_SMD:R_0603_1608Metric_Pad0.98x0.95mm_HandSolder, symbol Device:R
- added R65: 15k, Resistor_SMD:R_0603_1608Metric_Pad0.98x0.95mm_HandSolder, symbol Device:R
- added R66: 22K, Resistor_SMD:R_0603_1608Metric_Pad0.98x0.95mm_HandSolder, symbol Device:R
- added R67: 10k, Resistor_SMD:R_0603_1608Metric_Pad0.98x0.95mm_HandSolder, symbol Device:R
- added R68: 100K, Resistor_SMD:R_0603_1608Metric_Pad0.98x0.95mm_HandSolder, symbol Device:R
- added SW7: SW_Push_SPDT, Button_Switch_SMD:SW_SPDT_PCM12, symbol Switch:SW_Push_SPDT
- added TP8: TestPoint_Probe, TestPoint:TestPoint_Pad_D1.0mm, symbol Connector:TestPoint_Probe
- added U23: REGLETA, Package_TO_SOT_SMD:SOT-23-5_HandSoldering, symbol LIB_REGULADORES:ME6211C33_LINEAL
- added U24: MCU, Package_TO_SOT_SMD:SOT-23-5_HandSoldering, symbol LIB_REGULADORES:ME6211C33_LINEAL
- added U26: MSTPS563200DDCR, Package_TO_SOT_SMD:SOT-23-6, symbol LIB_REGULADORES:MSTPS563200DDCR_BUCK
- added U29: (no value), Footprint:BRIDGE_2P, symbol LIB_CONECTORES:BRIDGE_2P
- L1: value 4.7uH -> 3.3uH; footprint Inductor_SMD:L_Wuerth_HCM-7050 -> Inductor_SMD:L_Sunlord_MWSA0402S
- R57: value 100k -> 10k; footprint Resistor_SMD:R_0805_2012Metric_Pad1.20x1.40mm_HandSolder -> Resistor_SMD:R_0603_1608Metric_Pad0.98x0.95mm_HandSolder
Connections:
- net +3.3V: now also C43.1, U24.5 (VOUT); no longer C33.1
- net +3.3VA: now also C33.1, U23.5 (VOUT); no longer C43.1
- net +5V: now also L1.1, C47.1, C48.2, R64.1, TP8.1, U23.1 (VIN), U23.3 (CE), U24.1 (VIN), U24.3 (CE); no longer L1.2
- net GND: now also C46.2, C47.2, C48.1, C49.2, C50.1, C51.2, C52.1, D14.1 (K), J14.1 (GND), R66.2, SW7.2 (B), U23.2 (VSS), U24.2 (VSS), U26.1 (GND)
- net VBATT: now also C46.1, C49.1, C50.2, C51.1, C52.2, J6.5 (D1), J6.6 (D2), R63.2, R67.1, U26.3 (VIN), U29.2 (B)
- net at R57.1: now also D13.2 (A), J6.2 (G1), J6.4 (G2), R68.2
- net at R57.2: now also SW7.1 (A)
- new net: C45.2, L1.2, U26.2 (SW)
- new net: R64.2, R65.1
- new net: D13.1 (K), J14.2 (VCC), J6.1 (S1), J6.3 (S2), R68.1, U29.1 (A)
- new net: D14.2 (A), R67.2
- new net: R65.2, R66.1, U26.4 (FB)
- new net: R63.1, U26.5 (EN)
- new net: C45.1, U26.6 (BST)
