File: Inda_Kicad/Inda_Kicad.kicad_pcb (KiCad board)
At the start: 4 copper layers, 135 x 78.5 mm, 201 parts, among them J1 FFC, J10 Conn_01x02_Socket, J11 XT30_BATT, J12 SQJ951EP, J13 SQJ951EP, J14 XT30_LIPO, J6 Conn_01x02_Socket, J7 Motor_8520, J8 FFC, J9 Conn_01x02_Socket, Q1 AO3400A, Q2 AO3400A, SW1 SW_Push, SW2 SW_Push, SW3 SW_Push, SW4 SW_Push, SW5 SW_Push_SPDT, U1 vs1838, U10 QRE111GR, U11 QRE111GR, U12 QRE111GR, U13 QRE111GR, U14 QRE111GR, U15 QRE111GR, U16 CD74HC4067SM, U17 QRE111GR, U18 QRE111GR, U19 QRE111GR, U20 QRE111GR, U21 MP6551GQB-P, U22 AD8418, U23 AD8418, U24 MP6551GQB-P, U25 CN3903, U26 ME6211C33_regulador, U27 MT6701CT, U28 MT6701CT, U29 ME6211C33_regulador, U3 MPU6500, U4 QRE111GR, U5 QRE111GR, U6 QRE111GR, U7 QRE111GR, U8 QRE111GR, U9 QRE111GR, Y1 Crystal_GND24

Commit message: kicad cambios
Parts:
- removed D9: 12v, Diode_SMD:D_1206_3216Metric_Pad1.42x1.75mm_HandSolder
- removed J12: SQJ951EP, Package_SO:PowerPAK_SO-8_Dual
- removed J14: XT30_LIPO, Connector_AMASS:AMASS_XT30U-F_1x02_P5.0mm_Vertical
- removed J6: Conn_01x02_Socket, Connector_PinHeader_2.54mm:PinHeader_1x02_P2.54mm_Vertical
- removed R53, R54: 0.033, Resistor_SMD:R_2512_6332Metric_Pad1.40x3.35mm_HandSolder
- removed R55: 100k, Resistor_SMD:R_0805_2012Metric_Pad1.20x1.40mm_HandSolder
- removed U22, U23: AD8418, Footprint:AD8418_MicroSoic
- removed kibuzzard-69E2B1AE (x2): G***, kibuzzard-69E2B1AE
- removed kibuzzard-69E2B1FC: G***, kibuzzard-69E2B1FC
- removed kibuzzard-69E2B208: G***, kibuzzard-69E2B208
- removed kibuzzard-69E2B20B: G***, kibuzzard-69E2B20B
- removed kibuzzard-69E2B212: G***, kibuzzard-69E2B212
- removed kibuzzard-69E2B220: G***, kibuzzard-69E2B220
- removed kibuzzard-69E2B227: G***, kibuzzard-69E2B227
- removed kibuzzard-69E2B22F: G***, kibuzzard-69E2B22F
- removed kibuzzard-69E2B236: G***, kibuzzard-69E2B236
- removed kibuzzard-69E2B23E: G***, kibuzzard-69E2B23E
- removed kibuzzard-69E2B2B1 (x4): G***, kibuzzard-69E2B2B1
- removed kibuzzard-69E2B33D: G***, kibuzzard-69E2B33D
- removed kibuzzard-69E2B382: G***, kibuzzard-69E2B382
- removed kibuzzard-69E2B3C8: G***, kibuzzard-69E2B3C8
- removed kibuzzard-69E2B437: G***, kibuzzard-69E2B437
- removed kibuzzard-69E2B43D: G***, kibuzzard-69E2B43D
- added G***: LOGO, LOGO, F.Cu at (98.9, 73.5)
- C39, C41, J15, J16, JP1, JP2, R61, R62, SW1, SW4: moved to F.Cu
- R1, R10, R11, R12, R13, R14, R15, R16, R17, R18, R19, R2, R20, R21, R22, R23, R24, R25, R26, R27, R28, R29, R3, R30, R31, R32, R33, R34, R35, R36, R37, R38, R39, R4, R40, R41, R42, R43, R44, R45, R46, R47, R48, R49, R5, R50, R51, R52, R6, R7, R8, R9: footprint Resistor_SMD:R_0805_2012Metric_Pad1.20x1.40mm_HandSolder -> Resistor_SMD:R_0603_1608Metric_Pad0.98x0.95mm_HandSolder
- moved G*** 204.9 mm to (315.0, 99.5)
- moved G*** 166.0 mm to (236.5, 2.72)
- moved H8 139.2 mm to (218.6, 67.9)
- moved JP1 134.0 mm to (244.2, 41.3), turned to 0 degrees
- moved H7 133.4 mm to (218.6, 62.5)
- moved D2 133.4 mm to (202.9, 41.2)
- moved C24 130.4 mm to (226.3, 97.9), turned to 0 degrees
- moved C39 126.7 mm to (239.9, 40.8)
- moved R61 125.7 mm to (239.9, 45.8)
- moved D3 125.4 mm to (202.9, 44.6)
- moved J15 124.8 mm to (239.6, 53.8), turned to 0 degrees
- moved U27 120.6 mm to (233.5, 42.9), turned to 0 degrees
- moved J4 119.1 mm to (215.5, 75.4), turned to 0 degrees
- moved C25 115.9 mm to (226.3, 100.4), turned to 0 degrees
- moved C26 115.6 mm to (229.3, 85.4), turned to 0 degrees
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Connections:
- J13 pad 1: Net-(D9-K) -> Net-(J11-VCC)
- J13 pad 2: Net-(D9-A) -> Net-(J13-G1)
- J13 pad 3: Net-(D9-K) -> Net-(J11-VCC)
- J13 pad 4: Net-(D9-A) -> Net-(J13-G1)
- R57 pad 1: Net-(D9-K) -> Net-(J11-VCC)
- R57 pad 2: Net-(SW5-A) -> Net-(J13-G1)
- SW5 pad 1: Net-(SW5-A) -> Net-(J13-G1)
- U21 pad 1: /Motores/SHUNT_SENSOR_ML -> /Motores/MOTB_ML
- U21 pad 10: /Motores/SHUNT_SENSOR_ML -> /Motores/MOTB_ML
- U24 pad 3: /Motores/SHUNT_SENSOR_MR -> /Motores/MOTB_MR
- U24 pad 8: /Motores/SHUNT_SENSOR_MR -> /Motores/MOTB_MR
Routing:
- net /Sensores/3V3_MOD: track 469.4 -> 0.00 mm, vias 12 -> 0
- net /Sensores/GND_MOD: track 324.6 -> 0.00 mm, vias 29 -> 0
- net /MOTOR_EN: track 157.8 -> 0.00 mm, vias 7 -> 0
- net /SENSOR_A_ML: track 134.8 -> 0.00 mm, vias 4 -> 0
- net /VOLTAGE_BATT: track 112.8 -> 0.00 mm, vias 2 -> 0
- net +3.3V: track 103.4 -> 0.00 mm, vias 2 -> 0
- net /LED1: track 99.9 -> 0.00 mm, vias 4 -> 0
- net /ENCC_ML: track 98.6 -> 0.00 mm, vias 2 -> 0
- net /ENCB_ML: track 98.5 -> 0.00 mm, vias 2 -> 0
- net /ENCA_ML: track 93.7 -> 0.00 mm, vias 3 -> 0
- net /PWMA_ML: track 92.4 -> 0.00 mm, vias 2 -> 0
- net /LED2: track 92.2 -> 0.00 mm, vias 4 -> 0
- net /PWMB_ML: track 92.0 -> 0.00 mm, vias 2 -> 0
- net +3.3VA: track 77.8 -> 0.00 mm, vias 19 -> 0
- net GND: track 75.5 -> 0.00 mm, vias 70 -> 0
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- removed copper zone on In2.Cu, net +3.3VA
- removed copper zone on F.Cu, net /Motores/MOTA_ML
- removed copper zone on In2.Cu, net /Motores/MOTA_ML
- removed copper zone on F.Cu, net /Motores/MOTA_MR
- removed copper zone on In2.Cu, net /Motores/MOTA_MR
- removed copper zone on F.Cu, net /Motores/MOTB_ML
- removed copper zone on In2.Cu, net /Motores/MOTB_ML
- removed copper zone on F.Cu, net /Motores/MOTB_MR
- removed copper zone on In2.Cu, net /Motores/MOTB_MR
- removed copper zone on F.Cu, net /Motores/SHUNT_SENSOR_ML
- removed copper zone on In2.Cu, net /Motores/SHUNT_SENSOR_ML
- removed copper zone on F.Cu, net /Motores/SHUNT_SENSOR_MR
- removed copper zone on In2.Cu, net /Motores/SHUNT_SENSOR_MR
- removed copper zone on F.Cu, net /VOLTAGE
- removed copper zone on In2.Cu, net /VOLTAGE
- removed copper zone on F.Cu, net Net-(D9-A)
- removed copper zone on In2.Cu, net Net-(D9-A)
- removed copper zone on F.Cu, net Net-(J11-VCC)
- removed copper zone on In2.Cu, net Net-(J11-VCC)
- removed copper zone on F.Cu, net Net-(U25-SW)
