File: Inda_Kicad/Inda_Kicad.kicad_pcb (KiCad board)
At the start: 4 copper layers, 135 x 78.5 mm, 173 parts, among them J1 FFC, J10 Conn_01x02_Socket, J11 XT30_BATT, J13 SQJ951EP, J7 Motor_8520, J8 FFC, J9 Conn_01x02_Socket, Q1 AO3400A, Q2 AO3400A, SW1 SW_Push, SW2 SW_Push, SW3 SW_Push, SW4 SW_Push, SW5 SW_Push_SPDT, U1 vs1838, U10 QRE111GR, U11 QRE111GR, U12 QRE111GR, U13 QRE111GR, U14 QRE111GR, U15 QRE111GR, U16 CD74HC4067SM, U17 QRE111GR, U18 QRE111GR, U19 QRE111GR, U20 QRE111GR, U21 MP6551GQB-P, U24 MP6551GQB-P, U25 CN3903, U26 ME6211C33_regulador, U27 MT6701CT, U28 MT6701CT, U29 ME6211C33_regulador, U3 MPU6500, U4 QRE111GR, U5 QRE111GR, U6 QRE111GR, U7 QRE111GR, U8 QRE111GR, U9 QRE111GR, Y1 Crystal_GND24

Commit message: Seguidor V3 con turbina finalizado a espera de revision
Parts:
- removed C16, C5: 4.7uF, Capacitor_SMD:C_0603_1608Metric_Pad1.08x0.95mm_HandSolder
- removed C17: 1uF, Capacitor_SMD:C_0603_1608Metric_Pad1.08x0.95mm_HandSolder
- removed C2, C3, C4: 10nF, Capacitor_SMD:C_0603_1608Metric_Pad1.08x0.95mm_HandSolder
- removed C34: 100nF, Capacitor_SMD:C_0603_1608Metric_Pad1.08x0.95mm_HandSolder
- removed the G*** at (293.5, 85.5)
- removed SW4: SW_Push, Button_Switch_SMD:SW_Push_SPST_NO_Alps_SKRK
- removed SW5: SW_Push_SPDT, Button_Switch_SMD:SW_SPDT_PCM12
- added C38: 100nF, Capacitor_SMD:C_0603_1608Metric_Pad1.08x0.95mm_HandSolder, F.Cu at (107.2, 85.0)
- added C40: 1uF, Capacitor_SMD:C_0603_1608Metric_Pad1.08x0.95mm_HandSolder, F.Cu at (107.2, 86.8)
- added C45: 0.1uF, Capacitor_SMD:C_0603_1608Metric, F.Cu at (99.7, 124.7)
- added C46: 22uF, Capacitor_Tantalum_SMD:CP_EIA-3528-15_AVX-H_HandSolder, F.Cu at (106.7, 133.3)
- added C47: 22uF, Capacitor_Tantalum_SMD:CP_EIA-3528-15_AVX-H_HandSolder, F.Cu at (99.9, 122.1)
- added C48: 22uF, Capacitor_SMD:C_0603_1608Metric, F.Cu at (94.8, 122.0)
- added C49: 10uF, Capacitor_Tantalum_SMD:CP_EIA-3528-15_AVX-H_HandSolder, F.Cu at (112.5, 110.3)
- added C50: 100nF, Capacitor_SMD:C_0603_1608Metric, F.Cu at (109.6, 109.2)
- added C51: 10uF, Capacitor_Tantalum_SMD:CP_EIA-3528-15_AVX-H_HandSolder, F.Cu at (87.6, 110.3)
- added C52: 100nF, Capacitor_SMD:C_0603_1608Metric, F.Cu at (90.4, 109.2)
- added D11: LED, LED_SMD:LED_0805_2012Metric_Pad1.15x1.40mm_HandSolder, F.Cu at (109.0, 145.5)
- added D12: LED, LED_SMD:LED_0805_2012Metric_Pad1.15x1.40mm_HandSolder, F.Cu at (116.4, 92.2)
- added D13: 12V, Resistor_SMD:R_1206_3216Metric_Pad1.30x1.75mm_HandSolder, F.Cu at (92.8, 134.6)
- added D14: GREEN, LED_SMD:LED_1206_3216Metric_Pad1.42x1.75mm_HandSolder, B.Cu at (141.0, 129.0)
- added D15: LED, LED_SMD:LED_0805_2012Metric_Pad1.15x1.40mm_HandSolder, F.Cu at (110.8, 143.8)
- added D18: LED, LED_SMD:LED_1206_3216Metric_Pad1.42x1.75mm_HandSolder, F.Cu at (197.0, 80.5)
- added D19: BAT54A, Package_TO_SOT_SMD:SOT-23, F.Cu at (207.0, 88.0)
- added D20: LED, LED_SMD:LED_1206_3216Metric_Pad1.42x1.75mm_HandSolder, F.Cu at (207.0, 80.5)
- added D9: SS34, Diode_SMD:D_SMA, F.Cu at (120.0, 116.0)
- added H10: MountingHole_Pad, MountingHole:MountingHole_2.2mm_M2_ISO14580_Pad, F.Cu at (92.0, 13.0)
- added H11: MountingHole_Pad, Footprint:PAD_MOTOR_1725, F.Cu at (175.0, 156.5)
- added H12: MountingHole_Pad, Footprint:PAD_MOTOR_1725, F.Cu at (175.0, 143.5)
- added H13: MountingHole_Pad, Footprint:PAD_MOTOR_1725, F.Cu at (152.4, 158.3)
- added H14: MountingHole_Pad, Footprint:PAD_MOTOR_1725, F.Cu at (152.4, 145.3)
- added H9: MountingHole_Pad, MountingHole:MountingHole_2.2mm_M2_ISO14580_Pad, F.Cu at (108.0, 13.0)
- added J12: ENC_MR, Footprint:CONN_MT6701_THT_1.6mm_MALE, F.Cu at (144.3, 174.2)
- added J14: XT30, Footprint:XT30U-F_1x02_P5.0mm_Vertical, F.Cu at (102.5, 139.5)
- added J17: IN_IR_MR, Footprint:CONN_01X04_2IR_LINEA_FEMALE, F.Cu at (59.3, 83.8)
- added J18: MOTOR_ML, Connector_JST:JST_PH_S2B-PH-K_1x02_P2.00mm_Horizontal, F.Cu at (175.0, 151.0)
- added J19: MOTOR_MR, Connector_JST:JST_PH_S2B-PH-K_1x02_P2.00mm_Horizontal, F.Cu at (152.5, 152.8)
- added J3: MR, Connector_JST:JST_PH_B2B-PH-K_1x02_P2.00mm_Vertical, F.Cu at (125.8, 92.5)
- added J6: SQJ951EP, Package_SO:PowerPAK_SO-8_Dual, F.Cu at (101.0, 133.2)
- added Q3: AO3400A, Package_TO_SOT_SMD:SOT-23, F.Cu at (126.4, 116.0)
- added R53: 10k, Resistor_SMD:R_0603_1608Metric_Pad0.98x0.95mm_HandSolder, F.Cu at (129.6, 116.0)
- added R54: 100, Resistor_SMD:R_0603_1608Metric_Pad0.98x0.95mm_HandSolder, F.Cu at (131.6, 116.0)
- added R55: 100, Resistor_SMD:R_0603_1608Metric_Pad0.98x0.95mm_HandSolder, F.Cu at (68.2, 116.0)
- added R63: 200K, Resistor_SMD:R_0603_1608Metric_Pad0.98x0.95mm_HandSolder, F.Cu at (104.5, 124.7)
- added R64: 100k, Resistor_SMD:R_0603_1608Metric_Pad0.98x0.95mm_HandSolder, F.Cu at (106.5, 124.7)
- added R65: 15k, Resistor_SMD:R_0603_1608Metric_Pad0.98x0.95mm_HandSolder, F.Cu at (106.5, 128.2)
- added R66: 22K, Resistor_SMD:R_0603_1608Metric_Pad0.98x0.95mm_HandSolder, F.Cu at (104.5, 128.2)
- added R67: 10k, Resistor_SMD:R_0603_1608Metric_Pad0.98x0.95mm_HandSolder, F.Cu at (132.0, 120.0)
- added R68: 100K, Resistor_SMD:R_0603_1608Metric_Pad0.98x0.95mm_HandSolder, F.Cu at (93.4, 131.0)
- added R69: 220, Resistor_SMD:R_0603_1608Metric_Pad0.98x0.95mm_HandSolder, F.Cu at (108.6, 140.5)
- added R70: 18k, Resistor_SMD:R_0603_1608Metric_Pad0.98x0.95mm_HandSolder, B.Cu at (197.0, 78.5)
- added R71: 18k, Resistor_SMD:R_0603_1608Metric_Pad0.98x0.95mm_HandSolder, B.Cu at (207.0, 90.5)
- added R72: 100, Resistor_SMD:R_0603_1608Metric_Pad0.98x0.95mm_HandSolder, B.Cu at (197.0, 100.0)
- added R73: 100, Resistor_SMD:R_0603_1608Metric_Pad0.98x0.95mm_HandSolder, B.Cu at (207.0, 87.5)
- added R74: 18k, Resistor_SMD:R_0603_1608Metric_Pad0.98x0.95mm_HandSolder, B.Cu at (197.0, 90.5)
- added R75: 18k, Resistor_SMD:R_0603_1608Metric_Pad0.98x0.95mm_HandSolder, B.Cu at (207.0, 78.5)
- added R76: 10k, Resistor_SMD:R_0603_1608Metric_Pad0.98x0.95mm_HandSolder, F.Cu at (197.0, 91.5)
- added R78: 220, Resistor_SMD:R_0603_1608Metric_Pad0.98x0.95mm_HandSolder, F.Cu at (197.0, 84.5)
- added R80: 10k, Resistor_SMD:R_0603_1608Metric_Pad0.98x0.95mm_HandSolder, F.Cu at (207.0, 91.5)
- added R81: 220, Resistor_SMD:R_0603_1608Metric_Pad0.98x0.95mm_HandSolder, F.Cu at (207.0, 84.5)
- added SW7: SW_Push_SPDT, Button_Switch_SMD:SW_SPDT_PCM12, F.Cu at (59.5, 129.3)
- added TP10: TestPoint_Probe, TestPoint:TestPoint_Pad_D1.0mm, F.Cu at (72.5, 102.6)
- added TP11: TestPoint_Probe, TestPoint:TestPoint_Pad_D1.0mm, F.Cu at (130.4, 102.2)
- added TP12: TestPoint_Probe, TestPoint:TestPoint_Pad_D1.0mm, F.Cu at (137.9, 96.9)
- added TP13: TestPoint_Probe, TestPoint:TestPoint_Pad_D1.0mm, F.Cu at (122.2, 102.3)
- added TP16: TestPoint_Probe, TestPoint:TestPoint_Pad_D1.0mm, B.Cu at (98.2, 79.5)
- added TP5: TestPoint_Probe, TestPoint:TestPoint_Pad_D1.0mm, F.Cu at (80.0, 102.0)
- added TP8: TestPoint_Probe, TestPoint:TestPoint_Pad_D1.0mm, F.Cu at (90.2, 123.6)
- added TP9: TestPoint_Probe, TestPoint:TestPoint_Pad_D1.0mm, F.Cu at (70.2, 88.9)
- added U22: IRM-V838, Footprint:IRM-V838, F.Cu at (78.6, 81.2)
- added U23: REGLETA, Package_TO_SOT_SMD:SOT-23-5_HandSoldering, F.Cu at (106.8, 116.2)
- added U30: QRE111GR, Footprint:QRE1113GR_IR, B.Cu at (197.0, 83.0)
- added U31: QRE111GR, Footprint:QRE1113GR_IR, B.Cu at (207.0, 95.0)
- added U32: QRE111GR, Footprint:QRE1113GR_IR, B.Cu at (197.0, 95.0)
- added U33: QRE111GR, Footprint:QRE1113GR_IR, B.Cu at (207.0, 83.0)
- added U34: SN74LVC1G14DBV, Package_TO_SOT_SMD:SOT-23-5, F.Cu at (197.0, 100.0)
- added U35: SN74LVC1G14DBV, Package_TO_SOT_SMD:SOT-23-5, F.Cu at (207.0, 95.0)
- added U36: SN74LVC1G14DBV, Package_TO_SOT_SMD:SOT-23-5, F.Cu at (207.0, 100.0)
- added kibuzzard-6A90F0A5: G***, kibuzzard-6A90F0A5, F.Cu at (116.4, 87.8)
- added kibuzzard-6A90F0BB: G***, kibuzzard-6A90F0BB, F.Cu at (119.2, 91.0)
- added kibuzzard-6A90F0C9: G***, kibuzzard-6A90F0C9, F.Cu at (122.0, 87.8)
- added kibuzzard-6A90F0F9: G***, kibuzzard-6A90F0F9, F.Cu at (114.0, 81.6)
- added kibuzzard-6A90F119: G***, kibuzzard-6A90F119, F.Cu at (126.2, 81.6)
- added kibuzzard-6A90F136: G***, kibuzzard-6A90F136, F.Cu at (137.8, 129.2)
- added kibuzzard-6A925322: G***, kibuzzard-6A925322, F.Cu at (90.5, 125.2)
- added kibuzzard-6A925429: G***, kibuzzard-6A925429, F.Cu at (132.9, 102.9)
- added kibuzzard-6A9254A2: G***, kibuzzard-6A9254A2, F.Cu at (71.0, 87.5)
- added kibuzzard-6A9254AE: G***, kibuzzard-6A9254AE, F.Cu at (75.1, 102.7)
- added kibuzzard-6A9254B8: G***, kibuzzard-6A9254B8, F.Cu at (118.8, 102.9)
- added kibuzzard-6A9254B8: G***, kibuzzard-6A9254B8, F.Cu at (140.3, 97.0)
- added kibuzzard-6A925561: G***, kibuzzard-6A925561, F.Cu at (83.0, 103.0)
- added kibuzzard-6A9255C9: G***, kibuzzard-6A9255C9, B.Cu at (95.6, 79.6)
- C12: value 100nF -> 4.7uF
- C14: value 100nF -> 1uF
- C18, C19, C22: moved to F.Cu
- C23, C24, C39, C41, G***, JP1, JP2, R61, R62: moved to B.Cu
- C29: value 10uF -> 100nF; footprint Capacitor_Tantalum_SMD:CP_EIA-6032-15_Kemet-U_HandSolder -> Capacitor_SMD:C_0805_2012Metric_Pad1.18x1.45mm_HandSolder
- C30: footprint Capacitor_SMD:C_0603_1608Metric_Pad1.08x0.95mm_HandSolder -> Capacitor_SMD:C_0805_2012Metric_Pad1.18x1.45mm_HandSolder
- C31: value 100nF -> 47uF
- C35: value 100nF -> 2.2uF
- C36: value 22uF -> 2.2uF
- C37: value 100uF -> 100nF; footprint Capacitor_Tantalum_SMD:CP_EIA-6032-15_Kemet-U_HandSolder -> Capacitor_SMD:C_0603_1608Metric_Pad1.08x0.95mm_HandSolder
- D10: value LED -> BAT54C; footprint LED_SMD:LED_1206_3216Metric_Pad1.42x1.75mm_HandSolder -> Package_TO_SOT_SMD:SOT-23
- D2, D3, D4, D5, D6, D7: footprint LED_SMD:LED_1206_3216Metric_Pad1.42x1.75mm_HandSolder -> LED_SMD:LED_0805_2012Metric_Pad1.15x1.40mm_HandSolder
- J1, J8: value FFC -> ~
- J10: value Conn_01x02_Socket -> ML; footprint Connector_Molex:Molex_SL_171971-0002_1x02_P2.54mm_Vertical -> Connector_JST:JST_PH_B2B-PH-K_1x02_P2.00mm_Vertical
- J11: value XT30_BATT -> ENC_ML; footprint Connector_AMASS:AMASS_XT30U-F_1x02_P5.0mm_Vertical -> Footprint:CONN_MT6701_THT_1.6mm_MALE
- J13: value SQJ951EP -> 8052_A; footprint Package_SO:PowerPAK_SO-8_Dual -> Connector_JST:JST_PH_B2B-PH-K_1x02_P2.00mm_Vertical
- J15: value ~ -> IR_ML; footprint Footprint:AS5145_Mod -> Footprint:CONN_01X04_2IR_LINEA_MALE
- J16: value ~ -> IN_IR_ML; footprint Footprint:AS5145_Mod -> Footprint:CONN_01X04_2IR_LINEA_FEMALE
- J4: value ~ -> ENC_MR; footprint Footprint:AS5145_CONN_PCB -> Footprint:CONN_MT6701_THT_1.6mm_FEMALE
- J5: value ~ -> ENC_ML; footprint Footprint:AS5145_CONN_PCB -> Footprint:CONN_MT6701_THT_1.6mm_FEMALE
- J7: value Motor_8520 -> 8052_B; footprint Connector_PinHeader_2.54mm:PinHeader_1x02_P2.54mm_Vertical -> Connector_JST:JST_PH_B2B-PH-K_1x02_P2.00mm_Vertical
- J9: value Conn_01x02_Socket -> IR_ML; footprint Connector_Molex:Molex_SL_171971-0002_1x02_P2.54mm_Vertical -> Footprint:CONN_01X04_2IR_LINEA_MALE
- L1: value 4.7uH -> 3.3uH; footprint Inductor_SMD:L_Wuerth_HCM-7050 -> Inductor_SMD:L_Sunlord_MWSA0402S
- R5: value 100 -> 10
- R56: value 220 -> 100; footprint Resistor_SMD:R_0805_2012Metric_Pad1.20x1.40mm_HandSolder -> Resistor_SMD:R_0603_1608Metric_Pad0.98x0.95mm_HandSolder; moved to B.Cu
- R57: value 100k -> 10k; footprint Resistor_SMD:R_0805_2012Metric_Pad1.20x1.40mm_HandSolder -> Resistor_SMD:R_0603_1608Metric_Pad0.98x0.95mm_HandSolder
- R58: value 10K -> 100; footprint Resistor_SMD:R_0805_2012Metric_Pad1.20x1.40mm_HandSolder -> Resistor_SMD:R_0603_1608Metric_Pad0.98x0.95mm_HandSolder; moved to B.Cu
- R59: value 44K -> 220; footprint Resistor_SMD:R_0805_2012Metric_Pad1.20x1.40mm_HandSolder -> Resistor_SMD:R_0603_1608Metric_Pad0.98x0.95mm_HandSolder
- R60: value 10K -> 220; footprint Resistor_SMD:R_0805_2012Metric_Pad1.20x1.40mm_HandSolder -> Resistor_SMD:R_0603_1608Metric_Pad0.98x0.95mm_HandSolder
- SW1: value SW_Push -> nrst
- SW2: value SW_Push -> START
- SW3: value SW_Push -> STOP
- U1: value vs1838 -> SN74LVC1G14DBV; footprint Connector_PinHeader_2.54mm:PinHeader_1x03_P2.54mm_Vertical -> Package_TO_SOT_SMD:SOT-23-5
- U2: value ~ -> MP6551GQB-P; footprint Package_QFP:LQFP-64_10x10mm_P0.5mm -> Footprint:MP6551
- U24: value MP6551GQB-P -> MCU; footprint Footprint:MP6551 -> Package_TO_SOT_SMD:SOT-23-5_HandSoldering
- U25: value CN3903 -> 405RGT6; footprint Package_SO:HSOP-8-1EP_3.9x4.9mm_P1.27mm_EP2.41x3.1mm -> Package_QFP:LQFP-64_10x10mm_P0.5mm
- U26: value ME6211C33_regulador -> MSTPS563200DDCR; footprint Package_TO_SOT_SMD:SOT-23-5_HandSoldering -> Package_TO_SOT_SMD:SOT-23-6
- U29: value ME6211C33_regulador -> ~; footprint Package_TO_SOT_SMD:SOT-23-5_HandSoldering -> Footprint:BRIDGE_2P; moved to B.Cu
- moved G*** 247.9 mm to (68.3, 123.5)
- moved G*** 212.8 mm to (-111.5, 105.6)
- moved C39 168.9 mm to (130.9, 169.8), turned to 180 degrees
- moved JP1 166.8 mm to (132.8, 165.5)
- moved G*** 165.6 mm to (100.0, 14.0), turned to 180 degrees
- moved R61 163.6 mm to (130.9, 167.9), turned to 180 degrees
- moved C26 163.4 mm to (66.2, 94.8), turned to 90 degrees
- moved U27 160.2 mm to (132.8, 167.5)
- moved C25 160.1 mm to (66.2, 100.8), turned to 180 degrees
- moved C41 159.7 mm to (142.4, 169.8), turned to 180 degrees
- moved H4 159.0 mm to (59.0, 123.5)
- moved Q2 158.1 mm to (73.6, 116.0)
- moved U2 156.9 mm to (71.4, 98.2)
- moved JP2 156.6 mm to (144.3, 165.5)
- moved G*** 155.1 mm to (108.6, 90.4)
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Connections:
- net /Sensores/3V3_MOD renamed /SENSORES/3V3_MOD
- net /Sensores/GND_MOD renamed /SENSORES/GND_MOD
- net /Sensores/OUT0_IR_MOD renamed /SENSORES/OUT0_IR_MOD
- net /Sensores/OUT10_IR_MOD renamed /SENSORES/OUT10_IR_MOD
- net /Sensores/OUT11_IR_MOD renamed /SENSORES/OUT11_IR_MOD
- net /Sensores/OUT12_IR_MOD renamed /SENSORES/OUT12_IR_MOD
- net /Sensores/OUT13_IR_MOD renamed /SENSORES/OUT13_IR_MOD
- net /Sensores/OUT14_IR_MOD renamed /SENSORES/OUT14_IR_MOD
- net /Sensores/OUT15_IR_MOD renamed /SENSORES/OUT15_IR_MOD
- net /Sensores/OUT1_IR_MOD renamed /SENSORES/OUT1_IR_MOD
- net /Sensores/OUT2_IR_MOD renamed /SENSORES/OUT2_IR_MOD
- net /Sensores/OUT3_IR_MOD renamed /SENSORES/OUT3_IR_MOD
- net /Sensores/OUT4_IR_MOD renamed /SENSORES/OUT4_IR_MOD
- net /Sensores/OUT5_IR_MOD renamed /SENSORES/OUT5_IR_MOD
- net /Sensores/OUT6_IR_MOD renamed /SENSORES/OUT6_IR_MOD
- net /Sensores/OUT7_IR_MOD renamed /SENSORES/OUT7_IR_MOD
- net /Sensores/OUT8_IR_MOD renamed /SENSORES/OUT8_IR_MOD
- net /Sensores/OUT9_IR_MOD renamed /SENSORES/OUT9_IR_MOD
- net /Sensores/OUT_MOD renamed /SENSORES/OUT_MOD
- net /Sensores/S0_MOD renamed /SENSORES/S0_MOD
- net /Sensores/S1_MOD renamed /SENSORES/S1_MOD
- net /Sensores/S2_MOD renamed /SENSORES/S2_MOD
- net /Sensores/S3_MOD renamed /SENSORES/S3_MOD
- C23 pad 1: +3.3VA -> /SENSORES/3V3_IR_ML
- C23 pad 2: GND -> /SENSORES/GND_IR_ML
- C24 pad 1: +3.3V -> /SENSORES/3V3_IR_MR
- C24 pad 2: GND -> /SENSORES/GND_IR_MR
- C25 pad 1: /VOLTAGE -> /VOLTAJE
- C26 pad 1: /VOLTAGE -> /VOLTAJE
- C27 pad 1: /VOLTAGE -> /VOLTAJE
- C28 pad 1: /VOLTAGE -> /VOLTAJE
- C29 pad 1: /VOLTAGE -> Net-(J18-Pin_1)
- C29 pad 2: GND -> Net-(J18-Pin_2)
- C30 pad 1: /VOLTAGE -> Net-(J19-Pin_1)
- C30 pad 2: GND -> Net-(J19-Pin_2)
- C31 pad 1: Net-(U25-BST) -> +3.3VA
- C31 pad 2: Net-(U25-SW) -> GND
- C33 pad 1: +3.3V -> +3.3VA
- C35 pad 1: +5V -> Net-(U25-VCAP_2)
- C36 pad 1: +5V -> Net-(U25-VCAP_1)
- C37 pad 1: +5V -> +3.3VA
- C39 pad 1: /Encoder/VCCA_CONN -> /ENCODER/VCCA_CONN
- C39 pad 2: /Encoder/GNDA_CONN -> /ENCODER/GNDA_CONN
- C41 pad 1: /Encoder/VCCB_CONN -> /ENCODER/VCCB_CONN
- C41 pad 2: /Encoder/GNDB_CONN -> /ENCODER/GNDB_CONN
- C43 pad 1: +3.3VA -> +3.3V
- C7 pad 1: /OSC_A -> /OSC_B
- C9 pad 1: /OSC_B -> /OSC_A
- D10 pad 1: Net-(D10-K) -> /SENSORES/B_IR_ML
- D10 pad 2: /VOLTAGE -> /SENSORES/A_IR_ML
- D8 pad 1: /VOLTAGE -> /VOLTAJE
- J10 pad 1: /Motores/MOTB_MR -> /MOTOR/MOTB_ML
- J10 pad 2: /Motores/MOTA_MR -> /MOTOR/MOTA_ML
- J11 pad 1: GND -> /ENCODER/GNDA_CONN
- J11 pad 2: Net-(J11-VCC) -> /ENCODER/VCCA_CONN
- J13 pad 1: Net-(J11-VCC) -> /VOLTAJE
- J13 pad 2: Net-(J13-G1) -> Net-(D9-A)
- J15 pad 1: /Encoder/GNDA_CONN -> /SENSORES/GND_IR_MR
- J15 pad 2: /Encoder/VCCA_CONN -> /SENSORES/3V3_IR_MR
- J15 pad 3: /Encoder/ENCA_ML_CONN -> /SENSORES/OUT_IR_MR
- J15 pad 4: /Encoder/ENCB_ML_CONN -> /SENSORES/LED_IR_MR
- J16 pad 1: /Encoder/GNDB_CONN -> GND
- J16 pad 2: /Encoder/VCCB_CONN -> +3.3V
- J16 pad 3: /Encoder/ENCA_MR_CONN -> /IN_IR_ML
- J16 pad 4: /Encoder/ENCB_MR_CONN -> /LED_ML_LINEA
- J4 pad 2: +3.3V -> +3.3VA
- J4 pad 3: /ENCA_ML -> /ENCA_MR
- J4 pad 4: /ENCB_ML -> /ENCB_MR
- J4 pad 5: /ENCC_ML -> /ENCZ_MR
- J5 pad 3: /ENCA_MR -> /ENCA_ML
- J5 pad 4: /ENCB_MR -> /ENCB_ML
- J5 pad 5: /ENCC_MR -> /ENCZ_ML
- J7 pad 1: /VOLTAGE -> Net-(D8-A)
- J7 pad 2: Net-(D8-A) -> /VOLTAJE
- J9 pad 1: /Motores/MOTA_ML -> /SENSORES/GND_IR_ML
- J9 pad 2: /Motores/MOTB_ML -> /SENSORES/3V3_IR_ML
- JP1 pad 1: /Encoder/VCCA_CONN -> /ENCODER/VCCA_CONN
- JP2 pad 1: /Encoder/VCCB_CONN -> /ENCODER/VCCB_CONN
- L1 pad 1: Net-(U25-SW) -> +5V
- L1 pad 2: +5V -> Net-(U26-SW)
- Q2 pad 1: /PWM_MOTO_BRUSSHLES -> Net-(Q2-G)
- R15 pad 1: /VOLTAGE -> /VOLTAJE
- R19 pad 1: /PWM_MOTO_BRUSSHLES -> Net-(Q2-G)
- R3 pad 1: /BUTTON_STOP -> +3.3VA
- R3 pad 2: GND -> /BUTTON_STOP
- R5 pad 2: Net-(U1-vcc) -> Net-(U22-VCC)
- R56 pad 1: Net-(D10-K) -> /SENSORES/3V3_IR_ML
- R56 pad 2: GND -> Net-(U30-A)
- R57 pad 1: Net-(J11-VCC) -> Net-(D13-A)
- R57 pad 2: Net-(J13-G1) -> Net-(SW7-A)
- R58 pad 1: /VOLTAGE -> /SENSORES/3V3_IR_MR
- R58 pad 2: Net-(U25-EN) -> Net-(U31-A)
- R59 pad 1: /ALIMENTACION/FN -> Net-(D11-K)
- R59 pad 2: +5V -> GND
- R6 pad 1: /BUTTON_START -> +3.3VA
- R6 pad 2: GND -> /BUTTON_START
- R60 pad 1: GND -> Net-(D12-K)
- R60 pad 2: /ALIMENTACION/FN -> GND
- R61 pad 2: /Encoder/GNDA_CONN -> /ENCODER/GNDA_CONN
- R62 pad 2: /Encoder/GNDB_CONN -> /ENCODER/GNDB_CONN
- SW2 pad 1: +3.3VA -> /BUTTON_STOP
- SW2 pad 2: /BUTTON_STOP -> GND
- SW3 pad 1: +3.3VA -> /BUTTON_START
- SW3 pad 2: /BUTTON_START -> GND
- U1 pad 1: /IR_36KHZ -> unconnected-(U1-NC-Pad1)
- U1 pad 2: GND -> /SENSORES/IN_IR_ML
- U1 pad 3: Net-(U1-vcc) -> /SENSORES/GND_IR_ML
- U2 pad 1: +3.3VA -> /MOTOR/MOTB_ML
- U2 pad 10: /VOLTAGE_BATT -> /MOTOR/MOTB_ML
- U2 pad 11: /OUT_MUX -> unconnected-(U2-CM2-Pad11)
- U2 pad 12: GND -> unconnected-(U2-nFAULT-Pad12)
- U2 pad 13: +3.3VA -> /PWMA_ML
- U2 pad 14: /ENCA_MR -> /MOTOR_EN
- U2 pad 2: unconnected-(U2-PC13-Pad2) -> /VOLTAJE
- U2 pad 3: unconnected-(U2-PC14-OSC32_IN-Pad3) -> /MOTOR/MOTA_ML
- U2 pad 4: unconnected-(U2-PC15_OSC32_OUT-Pad4) -> /MOTOR_EN
- U2 pad 5: /OSC_A -> /PWMB_ML
- U2 pad 6: /OSC_B -> GND
- U2 pad 7: /NRST -> unconnected-(U2-CM1-Pad7)
- U2 pad 8: /SENSOR_A_MR -> /MOTOR/MOTA_ML
- U2 pad 9: /SENSOR_A_ML -> GND
- U21 pad 1: /Motores/MOTB_ML -> /MOTOR/MOTA_MR
- U21 pad 10: /Motores/MOTB_ML -> /MOTOR/MOTA_MR
- U21 pad 13: /PWMA_ML -> /PWMA_MR
- U21 pad 2: /VOLTAGE -> /VOLTAJE
- U21 pad 3: /Motores/MOTA_ML -> /MOTOR/MOTB_MR
- U21 pad 5: /PWMB_ML -> /PWMB_MR
- U21 pad 8: /Motores/MOTA_ML -> /MOTOR/MOTB_MR
- U24 pad 1: /Motores/MOTA_MR -> +5V
- U24 pad 2: /VOLTAGE -> GND
- U24 pad 3: /Motores/MOTB_MR -> +5V
- U24 pad 4: /MOTOR_EN -> unconnected-(U24-NC-Pad4)
- U24 pad 5: /PWMB_MR -> +3.3V
- U25 pad 1: Net-(U25-BST) -> +3.3VA
- U25 pad 2: /VOLTAGE -> /LED_OK
- U25 pad 3: Net-(U25-SW) -> /LED_ALARMA
- U25 pad 4: GND -> /LED_AVISO
- U25 pad 5: /ALIMENTACION/FN -> /OSC_A
- U25 pad 6: unconnected-(U25-NC-Pad6) -> /OSC_B
- U25 pad 7: Net-(U25-EN) -> /NRST
- U25 pad 8: unconnected-(U25-NC-Pad8) -> /OUT_MUX
- U25 pad 9: GND -> unconnected-(U25-PC1-Pad9)
- U26 pad 1: +5V -> GND
- U26 pad 2: GND -> Net-(U26-SW)
- U26 pad 3: +5V -> /VOLTAJE
- U26 pad 4: unconnected-(U26-NC-Pad4) -> Net-(U26-FB)
- U26 pad 5: +3.3V -> Net-(U26-EN)
- U27 pad 1: /Encoder/VCCA_CONN -> /ENCODER/VCCA_CONN
- U27 pad 4: /Encoder/GNDA_CONN -> /ENCODER/GNDA_CONN
- U27 pad 6: /Encoder/ENCA_ML_CONN -> /ENCODER/ENCA_ML_CONN
- U27 pad 7: /Encoder/ENCB_ML_CONN -> /ENCODER/ENCB_ML_CONN
- U27 pad 8: /Encoder/ENCC_ML_CONN -> /ENCODER/ENCC_ML_CONN
- U28 pad 1: /Encoder/VCCB_CONN -> /ENCODER/VCCB_CONN
- U28 pad 4: /Encoder/GNDB_CONN -> /ENCODER/GNDB_CONN
- U28 pad 6: /Encoder/ENCA_MR_CONN -> /ENCODER/ENCA_MR_CONN
- U28 pad 7: /Encoder/ENCB_MR_CONN -> /ENCODER/ENCB_MR_CONN
- U28 pad 8: /Encoder/ENCC_MR_CONN -> /ENCODER/ENCC_MR_CONN
- U29 pad 1: +5V -> Net-(D13-K)
- U29 pad 2: GND -> /VOLTAJE
- Y1 pad 1: /OSC_A -> /OSC_B
- Y1 pad 3: /OSC_B -> /OSC_A
Routing:
- net +3.3VA: track 0.00 -> 198.0 mm, vias 0 -> 17
- net /TX: track 0.00 -> 151.6 mm, vias 0 -> 4
- net /RX: track 0.00 -> 151.4 mm, vias 0 -> 2
- net /LED4: track 0.00 -> 140.7 mm, vias 0 -> 6
- net /LED5: track 0.00 -> 140.7 mm, vias 0 -> 6
- net /LED6: track 0.00 -> 140.4 mm, vias 0 -> 6
- net /SWCLK: track 0.00 -> 139.7 mm, vias 0 -> 4
- net /SWDIO: track 0.00 -> 138.6 mm, vias 0 -> 2
- net GND: track 0.00 -> 133.9 mm, vias 0 -> 83
- net /LED3: track 0.00 -> 120.9 mm, vias 0 -> 6
- net /LED2: track 0.00 -> 115.7 mm, vias 0 -> 6
- net /LED1: track 0.00 -> 113.2 mm, vias 0 -> 4
- net +3.3V: track 0.00 -> 96.5 mm, vias 0 -> 6
- net /PWM_Corelless_A: track 0.00 -> 91.4 mm, vias 0 -> 2
- net /NRST: track 0.00 -> 88.2 mm
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- added copper zone on F.Cu, net +3.3V
- added copper zone on In2.Cu, net +3.3V
- added copper zone on In2.Cu, net +3.3VA
- added copper zone on F.Cu, net +5V
- added copper zone on F.Cu, net /MOTOR/MOTA_ML
- added copper zone on In2.Cu, net /MOTOR/MOTA_ML
- added copper zone on F.Cu, net /MOTOR/MOTA_MR
- added copper zone on In2.Cu, net /MOTOR/MOTA_MR
- added copper zone on F.Cu, net /MOTOR/MOTB_ML
- added copper zone on In2.Cu, net /MOTOR/MOTB_ML
- added copper zone on F.Cu, net /MOTOR/MOTB_MR
- added copper zone on In2.Cu, net /MOTOR/MOTB_MR
- added copper zone on In2.Cu, net /SENSORES/3V3_IR_ML
- added copper zone on In2.Cu, net /SENSORES/3V3_IR_MR
- added copper zone on F.Cu, net /SENSORES/3V3_MOD
- added copper zone on In2.Cu, net /SENSORES/3V3_MOD
- added copper zone on In1.Cu, net /SENSORES/GND_IR_ML
- added copper zone on In1.Cu, net /SENSORES/GND_IR_MR
- added copper zone on F.Cu, net /SENSORES/GND_MOD
- added copper zone on In1.Cu, net /SENSORES/GND_MOD
- added copper zone on F.Cu, net /VOLTAJE
- added copper zone on In2.Cu, net /VOLTAJE
- added copper zone on In2.Cu, net GND
- added copper zone on F.Cu, net Net-(D13-K)
- added copper zone on In2.Cu, net Net-(D13-K)
- added copper zone on F.Cu, net Net-(Q1-D)
- added copper zone on F.Cu, net Net-(U26-SW)
Other:
- board size 135 x 78.5 mm -> 160 x 175.2 mm

Commit message: cambios en pcb y listo para mandar
Parts:
- removed the G*** at (-111.5, 105.6)
- added kibuzzard-6A97CCFF: G***, kibuzzard-6A97CCFF, B.Cu at (72.0, 115.5)
- G***: moved to B.Cu
- moved C41 149.7 mm to (98.1, 26.8)
- moved J12 149.7 mm to (100.0, 31.2)
- moved JP2 149.7 mm to (100.0, 22.5)
- moved R62 149.7 mm to (98.1, 24.9)
- moved U28 149.7 mm to (100.0, 24.5)
- moved C39 144.6 mm to (109.6, 26.8)
- moved J11 144.6 mm to (111.5, 31.2)
- moved R61 144.6 mm to (109.6, 24.9)
- moved U27 144.6 mm to (111.5, 24.5)
- moved JP1 144.6 mm to (111.5, 22.5)
- moved C24 130.9 mm to (88.7, 46.0)
- moved D19 130.9 mm to (88.7, 32.0)
- moved D20 130.9 mm to (88.7, 24.5)
- moved J15 130.9 mm to (88.7, 50.5)
- moved R58 130.9 mm to (88.7, 44.0)
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Other:
- board size 160 x 175.2 mm -> 100 x 155 mm
