File: Inda_Kicad/Inda_Kicad.kicad_sch (KiCad schematic)
At the start: 69 parts, among them J1 FFC, J6 Conn_01x02_Socket, J7 Motor_8520, Q1 AO3400A, Q2 AO3400A, SW1 SW_Push, SW2 SW_Push, SW3 SW_Push, SW4 SW_Push, U1 vs1838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

Commit message: kicad cambios
Parts:
- removed J6: Conn_01x02_Socket, Connector_PinHeader_2.54mm:PinHeader_1x02_P2.54mm_Vertical, symbol Connector:Conn_01x02_Socket
- R1, R10, R11, R12, R13, R14, R15, R16, R17, R18, R19, R2, R3, R4, R5, R6, R7, R8, R9: footprint Resistor_SMD:R_0805_2012Metric_Pad1.20x1.40mm_HandSolder -> Resistor_SMD:R_0603_1608Metric_Pad0.98x0.95mm_HandSolder
