File: Inda_Kicad/Inda_Kicad.kicad_sch (KiCad schematic)
At the start: 68 parts, among them J1 FFC, J7 Motor_8520, Q1 AO3400A, Q2 AO3400A, SW1 SW_Push, SW2 SW_Push, SW3 SW_Push, SW4 SW_Push, U1 vs1838, U3 MPU6500, Y1 Crystal_GND24

Commit message: Seguidor V3 con turbina finalizado a espera de revision
Parts:
- removed C16, C5: 4.7uF, Capacitor_SMD:C_0603_1608Metric_Pad1.08x0.95mm_HandSolder, symbol Device:C
- removed C17: 1uF, Capacitor_SMD:C_0603_1608Metric_Pad1.08x0.95mm_HandSolder, symbol Device:C
- removed C2, C3, C4: 10nF, Capacitor_SMD:C_0603_1608Metric_Pad1.08x0.95mm_HandSolder, symbol Device:C
- removed J1: FFC, Footprint:FFC_10x0.5, symbol Micromouse_Library:FFC_10X0.5
- removed J2: (no value), Footprint:usb_C_stm32, symbol Micromouse_Library:USB_C_SW_UART_CONECTOR
- removed J4, J5: (no value), Footprint:AS5145_CONN_PCB, symbol Micromouse_Library:CONN_5_PIN
- removed J7: Motor_8520, Connector_PinHeader_2.54mm:PinHeader_1x02_P2.54mm_Vertical, symbol Connector:Conn_01x02_Socket
- removed SW4: SW_Push, Button_Switch_SMD:SW_Push_SPST_NO_Alps_SKRK, symbol Switch:SW_Push
- removed U1: vs1838, Connector_PinHeader_2.54mm:PinHeader_1x03_P2.54mm_Vertical, symbol Micromouse_Library:1838
- removed U2: (no value), Package_QFP:LQFP-64_10x10mm_P0.5mm, symbol Micromouse_Library:STM32F401RCT6
- removed U3: MPU6500, Package_DFN_QFN:QFN-24-1EP_3x3mm_P0.4mm_EP1.75x1.6mm, symbol Micromouse_Library:MPU6500
- added C31: 47uF, Capacitor_SMD:C_0603_1608Metric_Pad1.08x0.95mm_HandSolder, symbol Device:C
- added C35, C36: 2.2uF, Capacitor_SMD:C_0603_1608Metric_Pad1.08x0.95mm_HandSolder, symbol Device:C
- added C37, C38: 100nF, Capacitor_SMD:C_0603_1608Metric_Pad1.08x0.95mm_HandSolder, symbol Device:C
- added C40: 1uF, Capacitor_SMD:C_0603_1608Metric_Pad1.08x0.95mm_HandSolder, symbol Device:C
- added D11, D12, D15: LED, LED_SMD:LED_0805_2012Metric_Pad1.15x1.40mm_HandSolder, symbol Device:LED
- added D9: SS34, Diode_SMD:D_SMA, symbol Diode:SS34
- added J1: (no value), Footprint:FFC_10x0.5, symbol LIB_CONECTORES:FFC_10X0.5
- added J13: 8052_A, Connector_JST:JST_PH_B2B-PH-K_1x02_P2.00mm_Vertical, symbol Connector_Generic:Conn_01x02
- added J16: IN_IR_ML, Footprint:CONN_01X04_2IR_LINEA_FEMALE, symbol Connector_Generic:Conn_01x04
- added J17: IN_IR_MR, Footprint:CONN_01X04_2IR_LINEA_FEMALE, symbol Connector_Generic:Conn_01x04
- added J2: (no value), Footprint:usb_C_stm32, symbol LIB_CONECTORES:USB_C_SW_UART_CONECTOR
- added J4: ENC_MR, Footprint:CONN_MT6701_THT_1.6mm_FEMALE, symbol Connector_Generic:Conn_01x05
- added J5: ENC_ML, Footprint:CONN_MT6701_THT_1.6mm_FEMALE, symbol Connector_Generic:Conn_01x05
- added J7: 8052_B, Connector_JST:JST_PH_B2B-PH-K_1x02_P2.00mm_Vertical, symbol Connector_Generic:Conn_01x02
- added Q3: AO3400A, Package_TO_SOT_SMD:SOT-23, symbol Transistor_FET:AO3400A
- added R53: 10k, Resistor_SMD:R_0603_1608Metric_Pad0.98x0.95mm_HandSolder, symbol Device:R
- added R54, R55: 100, Resistor_SMD:R_0603_1608Metric_Pad0.98x0.95mm_HandSolder, symbol Device:R
- added R59, R60, R69: 220, Resistor_SMD:R_0603_1608Metric_Pad0.98x0.95mm_HandSolder, symbol Device:R
- added TP16, TP5: TestPoint_Probe, TestPoint:TestPoint_Pad_D1.0mm, symbol Connector:TestPoint_Probe
- added U22: IRM-V838, Footprint:IRM-V838, symbol LIB_Componentes:IRM-V838
- added U25: 405RGT6, Package_QFP:LQFP-64_10x10mm_P0.5mm, symbol LIB_MCU:STM32F405RGT6
- added U3: MPU6500, Package_DFN_QFN:QFN-24-1EP_3x3mm_P0.4mm_EP1.75x1.6mm, symbol LIB_Componentes:MPU6500
- C12: value 100nF -> 4.7uF
- C14: value 100nF -> 1uF
- D2, D3, D4, D5, D6, D7: footprint LED_SMD:LED_1206_3216Metric_Pad1.42x1.75mm_HandSolder -> LED_SMD:LED_0805_2012Metric_Pad1.15x1.40mm_HandSolder
- R5: value 100 -> 10
- SW1: value SW_Push -> nrst
- SW2: value SW_Push -> START
- SW3: value SW_Push -> STOP
Connections:
- net +3.3V: now also J1.10, J1.9, J16.2 (Pin_2), J17.2 (Pin_2)
- net +3.3VA: now also R3.1, R6.1, C31.1, C37.1, C38.1, C40.1, J2.11 (VCC), J2.2 (VCC), J4.2 (Pin_2), J5.2 (Pin_2), U25.1 (VBAT), U25.13 (VDDA), U25.19 (VDD), U25.32 (VDD), U25.48 (VDD), U25.64 (VDD), U3.13 (VDD), U3.8 (VDDIO); no longer SW2.1, SW3.1
- net BOOT0: now also U25.60 (BOOT0)
- net BUTTON_START: now also R6.2, SW3.1, U25.24 (PC4); no longer R6.1, SW3.2
- net BUTTON_STOP: now also R3.2, SW2.1, U25.25 (PC5); no longer R3.1, SW2.2
- net ENCA_ML: now also J5.3 (Pin_3), U25.21 (PA5)
- net ENCA_MR: now also J4.3 (Pin_3), U25.14 (PA0)
- net ENCB_ML: now also J5.4 (Pin_4), U25.55 (PB3)
- net ENCB_MR: now also J4.4 (Pin_4), U25.15 (PA1)
- net EN_SENSORES: now also U25.37 (PC6)
- net GND: now also SW2.2, SW3.2, C31.2, C35.2, C36.2, C37.2, C38.2, C40.2, J16.1 (Pin_1), J17.1 (Pin_1), J2.1 (GND), J2.12 (GND), J2.13 (SHIELD), J4.1 (Pin_1), J5.1 (Pin_1), Q3.2 (S), R53.2, R59.2, R60.2, R69.2, U22.1 (GND), U22.4 (GND), U25.12 (VSSA), U25.18 (VSS), U25.63 (VSS), U3.18 (GND), U3.20 (RESV), U3.25 (EPAD); no longer R3.2, R6.2
- net IR_36KHZ: now also U22.3 (OUT), U25.45 (PA12)
- net LED1: now also U25.34 (PB13)
- net LED2: now also U25.33 (PB12)
- net LED3: now also U25.30 (PB11)
- net LED4: now also U25.29 (PB10)
- net LED_ALARMA: now also U25.3 (PC14)
- net LED_OK: now also U25.2 (PC13)
- net MISO: now also U25.52 (PC11), U3.9 (ADO/SDO)
- net MOSI: now also U25.53 (PC12), U3.24 (SDA/SDI)
- net MOTOR_EN: now also U25.57 (PB5)
- net NRST: now also U25.7 (NRST)
- net OSC_A: now also C9.1, Y1.3, U25.5 (PH0/OSC_IN); no longer C7.1, Y1.1
- net OSC_B: now also C7.1, Y1.1, U25.6 (PH1/OSC_OUT); no longer C9.1, Y1.3
- net OUT_MUX: now also J1.3, TP16.1, U25.8 (PC0)
- net PWMA_ML: now also U25.58 (PB6)
- net PWMA_MR: now also U25.62 (PB9)
- net PWMB_ML: now also U25.59 (PB7)
- net PWMB_MR: now also U25.61 (PB8)
- net PWM_BLUE: now also U25.22 (PA6)
- net PWM_GREEN: now also U25.23 (PA7)
- net PWM_RED: now also U25.26 (PB0)
- net RX: now also J2.10 (RX), J2.3 (RX), U25.43 (PA10)
- net S0_MUX: now also J1.4, U25.38 (PC7)
- net S1_MUX: now also J1.5, U25.39 (PC8)
- net S2_MUX: now also J1.7, U25.41 (PA8)
- net S3_MUX: now also J1.6, U25.40 (PC9)
- net SCK: now also U25.51 (PC10), U3.23 (SCL/SCLK)
- net SS: now also U25.50 (PA15), U3.22 (nCS)
- net SWCLK: now also J2.5 (SWCLK), J2.8 (SWCLK), U25.49 (PA14)
- net SWDIO: now also J2.6 (SWDIO), J2.7 (SWDIO), U25.46 (PA13)
- net TX: now also J2.4 (TX), J2.9 (TX), U25.42 (PA9)
- net VOLTAGE_BATT: now also TP5.1, U25.11 (PC3)
- net at D8.2 (A), Q2.3 (D): now also J7.1 (Pin_1)
- net at R5.2: now also U22.2 (VCC)
- net at Q1.3 (D): now also J1.1, J1.2
- net at C8.1: now also U3.10 (REGOUT)
- net PWM_MOTO_BRUSSHLES: no longer names the net of Q2.1 (G), R19.1
- net PWM_MOTO_BRUSSHLES: now also R55.2
- net VOLTAGE renamed VOLTAJE
- net VOLTAJE: now also D9.1 (K), J13.1 (Pin_1), J7.2 (Pin_2)
- new net: Q3.1 (G), R53.1, R54.2
- new net: D15.1 (K), R69.1
- new net: D12.1 (K), R60.1
- new net: C36.1, U25.31 (VCAP_1)
- new net: C35.1, U25.47 (VCAP_2)
- new net: D11.1 (K), R59.1
- new net: D9.2 (A), J13.2 (Pin_2), Q3.3 (D)
- new net ENCZ_ML: J5.5 (Pin_5), U25.56 (PB4)
- new net ENCZ_MR: J4.5 (Pin_5), U25.16 (PA2)
- new net IN_IR_ML: J16.3 (Pin_3), U25.44 (PA11)
- new net IN_IR_MR: J17.3 (Pin_3), U25.17 (PA3)
- new net LED5: D11.2 (A), U25.28 (PB2/BOOT1)
- new net LED6: D15.2 (A), U25.27 (PB1)
- new net LED_AVISO: D12.2 (A), U25.4 (PC15)
- new net LED_ML_LINEA: J16.4 (Pin_4), U25.54 (PD2)
- new net LED_MR_LINEA: J17.4 (Pin_4), U25.20 (PA4)
- new net PWM_Corelless_A: R54.1, U25.36 (PB15)
- new net PWM_Corelless_B: R55.1, U25.35 (PB14)
- no-connect marks 13 -> 8
Other:
- sheet Encoder renamed ENCODER
- sheet Motores renamed MOTOR
- sheet Sensores renamed SENSORES
- sheet MOTOR ports: added none; removed SENSOR_A_ML, SENSOR_A_MR
- moved on the sheet: C1, C10, C11, C12, C13, C14, C15, C44, C6, C7, C8, C9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
