File: Inda_Kicad/Motores.kicad_sch (KiCad schematic)
At the start: 14 parts, among them J10 Conn_01x02_Socket, J9 Conn_01x02_Socket, U21 MP6551GQB-P, U22 AD8418, U23 AD8418, U24 MP6551GQB-P

Commit message: kicad cambios
Parts:
- removed R53, R54: 0.033, Resistor_SMD:R_2512_6332Metric_Pad1.40x3.35mm_HandSolder, symbol Device:R
- removed U22, U23: AD8418, Footprint:AD8418_MicroSoic, symbol MOTORES_DRIVERS:AD8418
Connections:
- net SHUNT_SENSOR_ML is gone; now on net MOTB_ML: U21.1 (OUT1), U21.10 (OUT1)
- net SHUNT_SENSOR_MR is gone; now on net MOTB_MR: U24.3 (OUT2), U24.8 (OUT2)
- no-connect marks 8 -> 6
