File: Inda_Kicad/Motores.kicad_sch (KiCad schematic)
At the start: 10 parts, among them J10 Conn_01x02_Socket, J9 Conn_01x02_Socket, U21 MP6551GQB-P, U24 MP6551GQB-P

Commit message: Seguidor V3 con turbina finalizado a espera de revision
Parts:
- removed C23, C24: 100nF, Capacitor_SMD:C_0603_1608Metric_Pad1.08x0.95mm_HandSolder, symbol Device:C
- removed J10, J9: Conn_01x02_Socket, Connector_Molex:Molex_SL_171971-0002_1x02_P2.54mm_Vertical, symbol Connector:Conn_01x02_Socket
- removed U21, U24: MP6551GQB-P, Footprint:MP6551, symbol MOTORES_DRIVERS:MP6551GQB-P
- added C29, C30: 100nF, Capacitor_SMD:C_0805_2012Metric_Pad1.18x1.45mm_HandSolder, symbol Device:C
- added H11, H12, H13, H14: MountingHole_Pad, Footprint:PAD_MOTOR_1725, symbol Mechanical:MountingHole_Pad
- added J10: ML, Connector_JST:JST_PH_B2B-PH-K_1x02_P2.00mm_Vertical, symbol Connector_Generic:Conn_01x02
- added J18: MOTOR_ML, Connector_JST:JST_PH_S2B-PH-K_1x02_P2.00mm_Horizontal, symbol Connector_Generic:Conn_01x02
- added J19: MOTOR_MR, Connector_JST:JST_PH_S2B-PH-K_1x02_P2.00mm_Horizontal, symbol Connector_Generic:Conn_01x02
- added J3: MR, Connector_JST:JST_PH_B2B-PH-K_1x02_P2.00mm_Vertical, symbol Connector_Generic:Conn_01x02
- added TP10, TP11, TP12, TP13, TP9: TestPoint_Probe, TestPoint:TestPoint_Pad_D1.0mm, symbol Connector:TestPoint_Probe
- added U2, U21: MP6551GQB-P, Footprint:MP6551, symbol LIB_DRIVERS_MOTOR:MP6551GQB-P
Connections:
- net BATT: now also U2.2 (VBATT), U21.2 (VBATT)
- net EN_MOTOR: now also TP11.1, U2.14 (EN1), U2.4 (EN2), U21.14 (EN1), U21.4 (EN2)
- net GND: now also U2.6 (SR), U2.9 (GND), U21.6 (SR), U21.9 (GND)
- net MOTA_ML: now also J10.2 (Pin_2), U2.3 (OUT2), U2.8 (OUT2)
- net MOTA_MR: now also J3.1 (Pin_1), U21.1 (OUT1), U21.10 (OUT1)
- net MOTB_ML: now also J10.1 (Pin_1), U2.1 (OUT1), U2.10 (OUT1)
- net MOTB_MR: now also J3.2 (Pin_2), U21.3 (OUT2), U21.8 (OUT2)
- net PWMA_ML: now also TP9.1, U2.13 (IN_1)
- net PWMA_MR: now also TP13.1, U21.13 (IN_1)
- net PWMB_ML: now also TP10.1, U2.5 (IN2)
- net PWMB_MR: now also TP12.1, U21.5 (IN2)
- new net: C29.1, H11.1, J18.1 (Pin_1)
- new net: C29.2, H12.1, J18.2 (Pin_2)
- new net: C30.1, H13.1, J19.1 (Pin_1)
- new net: C30.2, H14.1, J19.2 (Pin_2)
