File: Inda_Kicad/Sensores.kicad_sch (KiCad schematic)
At the start: 56 parts, among them J8 FFC, U10 QRE111GR, U11 QRE111GR, U12 QRE111GR, U13 QRE111GR, U14 QRE111GR, U15 QRE111GR, U16 CD74HC4067SM, U17 QRE111GR, U18 QRE111GR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

Commit message: kicad cambios
Parts:
- R20, R21, R22, R23, R24, R25, R26, R27, R28, R29, R30, R31, R32, R33, R34, R35, R36, R37, R38, R39, R40, R41, R42, R43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: footprint Resistor_SMD:R_0805_2012Metric_Pad1.20x1.40mm_HandSolder -> Resistor_SMD:R_0603_1608Metric_Pad0.98x0.95mm_HandSolder
