File: Inda_Kicad/Sensores.kicad_sch (KiCad schematic)
At the start: 56 parts, among them J8 FFC, U10 QRE111GR, U11 QRE111GR, U12 QRE111GR, U13 QRE111GR, U14 QRE111GR, U15 QRE111GR, U16 CD74HC4067SM, U17 QRE111GR, U18 QRE111GR, U19 QRE111GR, U20 QRE111GR, U4 QRE111GR, U5 QRE111GR, U6 QRE111GR, U7 QRE111GR, U8 QRE111GR, U9 QRE111GR

Commit message: Seguidor V3 con turbina finalizado a espera de revision
Parts:
- removed J8: FFC, Footprint:FFC_10x0.5, symbol Micromouse_Library:FFC_10X0.5
- added C23, C24: 100nF, Capacitor_SMD:C_0603_1608Metric_Pad1.08x0.95mm_HandSolder, symbol Device:C
- added D10: BAT54C, Package_TO_SOT_SMD:SOT-23, symbol Diode:BAT54C
- added D18, D20: LED, LED_SMD:LED_1206_3216Metric_Pad1.42x1.75mm_HandSolder, symbol Device:LED
- added D19: BAT54A, Package_TO_SOT_SMD:SOT-23, symbol Diode:BAT54A
- added H10, H9: MountingHole_Pad, MountingHole:MountingHole_2.2mm_M2_ISO14580_Pad, symbol Mechanical:MountingHole_Pad
- added J15, J9: IR_ML, Footprint:CONN_01X04_2IR_LINEA_MALE, symbol Connector_Generic:Conn_01x04
- added J8: (no value), Footprint:FFC_10x0.5, symbol LIB_CONECTORES:FFC_10X0.5
- added R56, R58, R72, R73: 100, Resistor_SMD:R_0603_1608Metric_Pad0.98x0.95mm_HandSolder, symbol Device:R
- added R70, R71, R74, R75: 18k, Resistor_SMD:R_0603_1608Metric_Pad0.98x0.95mm_HandSolder, symbol Device:R
- added R76, R80: 10k, Resistor_SMD:R_0603_1608Metric_Pad0.98x0.95mm_HandSolder, symbol Device:R
- added R78, R81: 220, Resistor_SMD:R_0603_1608Metric_Pad0.98x0.95mm_HandSolder, symbol Device:R
- added U1, U34, U35, U36: SN74LVC1G14DBV, Package_TO_SOT_SMD:SOT-23-5, symbol 74xGxx:SN74LVC1G14DBV
- added U30, U31, U32, U33: QRE111GR, Footprint:QRE1113GR_IR, symbol LIB_Componentes:QRE1113GR
- U10, U11, U12, U13, U14, U15, U17, U18, U19, U20, U4, U5, U6, U7, U8, U9: symbol Micromouse_Library:QRE1113GR -> LIB_Componentes:QRE1113GR
Connections:
- net 3V3_MOD: now also J8.1, J8.2
- net GND_MOD: now also H10.1, H9.1, J8.10, J8.9
- net OUT_MOD: now also J8.8
- net S0_MOD: now also J8.7
- net S1_MOD: now also J8.6
- net S2_MOD: now also J8.4
- net S3_MOD: now also J8.5
- new net: R72.2, U32.1 (A)
- new net: D20.1 (K), R81.1
- new net: R56.2, U30.1 (A)
- new net: R58.2, U31.1 (A)
- new net: R73.2, U33.1 (A)
- new net: U1.4, U34.2
- new net: U35.4, U36.2
- new net: D18.1 (K), R78.1
- new net 3V3_IR_ML: C23.1, J9.2 (Pin_2), R56.1, R70.1, R72.1, R74.1, U1.5 (VCC), U34.5 (VCC)
- new net 3V3_IR_MR: C24.1, J15.2 (Pin_2), R58.1, R71.1, R73.1, R75.1, R80.2, U35.5 (VCC), U36.5 (VCC)
- new net A_IR_ML: D10.2, R70.2, U30.3
- new net A_IR_MR: D19.1, R71.2, U31.3
- new net B_IR_ML: D10.1, R74.2, U32.3
- new net B_IR_MR: D19.2, R75.2, U33.3
- new net GND_IR_ML: C23.2, J9.1 (Pin_1), R76.2, R78.2, U1.3 (GND), U30.2 (K), U30.4, U32.2 (K), U32.4, U34.3 (GND)
- new net GND_IR_MR: C24.2, J15.1 (Pin_1), R81.2, U31.2 (K), U31.4, U33.2 (K), U33.4, U35.3 (GND), U36.3 (GND)
- new net IN_IR_ML: D10.3, R76.1, U1.2
- new net IN_IR_MR: D19.3, R80.1, U35.2
- new net LED_IR_ML: D18.2 (A), J9.4 (Pin_4)
- new net LED_IR_MR: D20.2 (A), J15.4 (Pin_4)
- new net OUT_IR_ML: J9.3 (Pin_3), U34.4
- new net OUT_IR_MR: J15.3 (Pin_3), U36.4
Other:
- moved on the sheet: C18, C19, C20, C21, C22, R20, R21, R22, R23, R24, R25, R26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
